File: pcb/atx_power_control.brd (EAGLE design)
At the start: 30 x 30 mm, 25 parts, among them IC3 STM32F042F4, SW3 324_SW, SW4 324_SW, U2 USBC_16P, U4 XC6206_DEV

Commit message: working on PCB
Parts:
- removed JP1: (no value), pmm:PINHEAD_2X04
- removed R7: 1K, SparkFun-Passives:0805
- removed TP1, TP2, TP3, TP4, TP5: TPSQTP10SQ, testpad:TP10SQ
- removed U4: XC6206_DEV, 3pos_slide_switch:SOT23R_INFINEON
- added C3: 2.2uF, clock:0805@1
- added C5: 1uF, clock:0805@1
- added D3: (no value), adafruit:SOD-123FL
- added F1, F2, F3: FUSEX20MM, atx_power_control:FUSE_5MM
- added IC2: REG1117, clock:SOT223
- added IC4: MY_7905DT, atx_power_control:ADAFRUIT_TO252
- added J1: ATX24RH, SparkFun-Connectors:ATX24_RIGHT_ANGLE
- added J2, J3, J4, J5, J6, J7: (no value), SparkFun-Connectors:SCREWTERMINAL-3.5MM-2
- added U$1, U$10, U$2, U$3: M3_MOUNTING_HOLE, a:M3_MOUNTING_HOLE_PACK
- moved C2 103.9 mm to (122.6, 25.3)
- moved R6 103.9 mm to (107.3, 41.5)
- moved C1 103.9 mm to (125.7, 45.8)
- moved C4 103.9 mm to (125.7, 39.8)
- moved IC3 103.9 mm to (117.4, 23.5)
- moved JP3 103.9 mm to (129.9, 34.5)
- moved LED1 103.9 mm to (107.4, 36.5)
- moved LED2 103.9 mm to (107.4, 43.5)
- moved LED3 103.9 mm to (107.4, 29.5)
- moved R1 103.9 mm to (113.5, 37.7)
- moved R2 103.9 mm to (121.7, 37.7)
- moved R3 103.9 mm to (107.4, 27.5)
- moved R4 103.9 mm to (107.4, 34.5)
- moved R5 103.9 mm to (111.9, 22.5)
- moved SW3 103.9 mm to (127.4, 22.5)
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Connections:
- removed net +5V: C1.2, U2.A4B9, U2.B4A9, U4.3
- removed net N$15: IC3.10, TP5.TP
- removed net SCL: IC3.3, JP1.5, JP1.6
- new net VCC: C1.2, D3.C, IC2.3, J1.9
- net +3V3: now also IC2.2, IC2.4; no longer R7.2, U4.2
- net GND: now also C3.1, C5.1, IC2.1, IC4.1, J1.15, J1.17, J1.18, J1.19, J1.24, J1.3, J1.5, J1.7, J5.1, J5.2; no longer JP1.7, JP1.8, U4.1
- net N$10: now also D3.A, U2.A4B9, U2.B4A9; no longer JP1.1, JP1.2, R7.1
- net N$11: now also C5.2, IC4.2, J4.1, J4.2; no longer IC3.13, TP4.TP
- net N$12: now also J1.1, J1.12, J1.13, J1.2; no longer IC3.12, TP3.TP
- net N$13: now also F2.3, F2.4, J1.10, J1.11; no longer IC3.11, TP2.TP
- net N$14: now also F2.1, F2.2, J6.1, J6.2; no longer IC3.14, TP1.TP
- net N$2: now also C3.2, IC4.3, J1.14, J3.1, J3.2; no longer IC3.2, JP1.3, JP1.4
Routing:
- net N$6: track 37.3 -> 0.00 mm
- net +3V3: track 27.5 -> 0.00 mm, vias 6 -> 0
- net N$7: track 27.3 -> 0.00 mm
- net N$8: track 23.8 -> 0.00 mm, vias 2 -> 0
- net USB_DP: track 21.9 -> 0.00 mm
- net BUTTON1: track 19.9 -> 0.00 mm
- net USB_DN: track 19.9 -> 0.00 mm
- net +5V: track 19.0 -> 0.00 mm
- net N$9: track 18.0 -> 0.00 mm, vias 2 -> 0
- net N$4: track 16.7 -> 0.00 mm, vias 1 -> 0
- net SCL: track 12.2 -> 0.00 mm
- net N$3: track 11.8 -> 0.00 mm, vias 1 -> 0
- net BUTTON2: track 11.6 -> 0.00 mm
- net N$2: track 10.4 -> 0.00 mm
- net N$10: track 8.32 -> 0.00 mm
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Other:
- board size 30 x 30 mm -> 100 x 70 mm
- board text removed: "Bob Dishwasher Cassette Rewinder"
- board text removed: "CART OK"
- board text removed: "DONE"
- board text removed: "GND"
- board text removed: "POWER"
- board text removed: "RENEW"
- board text removed: "RESET"
- board text removed: "SCL"
- board text removed: "SDA"
- board text removed: "VCC"
- board text removed: "dekuNukem 2021"
- board text removed: "git.io/bob_rewind"
