File: pcb/atx_power_control.brd (EAGLE design)
At the start: 100 x 70 mm, 36 parts, among them IC2 REG1117, IC3 STM32F042F4, IC4 MY_7905DT, J1 ATX24RH, SW3 324_SW, SW4 324_SW, U2 USBC_16P

Commit message: working on PCB
Parts:
- removed D3: (no value), adafruit:SOD-123FL
- added C27: 47uF, clock:C1210
- added IC1: (no value), linear:TO220H
- added LED4, LED5, LED6, LED7: (no value), adafruit:CHIP-LED0805
- added R10, R8, R9: 1K, SparkFun-Passives:0805
- added R7: 5K, SparkFun-Passives:0805
- moved JP3 97.9 mm to (34.3, 55.8), turned to 0 degrees
- moved IC3 81.2 mm to (38.7, 43.7), turned to 0 degrees
- moved LED1 34.2 mm to (84.1, 11.4)
- moved R4 31.0 mm to (84.1, 14.0)
- moved IC2 10.7 mm to (24.9, 64.6), turned to 90 degrees
- moved IC4 5.68 mm to (30.7, 5.84)
- moved C3 5.34 mm to (27.9, 11.4)
- moved C5 5.24 mm to (33.5, 11.4)
- moved F1 3.81 mm to (69.6, 39.4), turned to 270 degrees
- moved F2 3.81 mm to (69.6, 48.3)
- moved F3 3.81 mm to (69.6, 30.5), turned to 270 degrees
- moved U2 2.03 mm to (38.7, 66.2)
Connections:
- new net N$15: F1.3, F1.4, J7.1, J7.2, LED7.A
- new net N$16: F3.3, F3.4, J2.1, J2.2, LED6.A
- new net N$18: LED6.C, R9.2
- new net N$20: LED7.C, R10.2
- net +3V3: no longer LED1.A
- net GND: now also C27.2, IC1.1, LED1.A, LED4.A, R10.1, R8.1, R9.1
- net N$10: now also F1.1, F1.2, J1.21, J1.22, J1.23, J1.4, J1.6; no longer D3.A, U2.A4B9, U2.B4A9
- net N$11: now also IC1.3, R4.1
- net N$12: now also F3.1, F3.2
- net N$14: now also LED5.A
- net N$2: now also C27.1, IC1.2, R7.1
- net N$8: now also LED4.C, R7.2; no longer IC3.6, R4.1
- net N$9: now also LED5.C, R8.2; no longer IC3.7, R3.1
- net VCC: now also U2.A4B9, U2.B4A9; no longer D3.C
Other:
- board text added: "-5V"

Commit message: working on PCB
Parts:
- removed J5: (no value), SparkFun-Connectors:SCREWTERMINAL-3.5MM-2
- added J10, J8, J9: (no value), SparkFun-Connectors:SCREWTERMINAL-3.5MM-2
- added JP1, JP2, JP7, JP8: (no value), pinhead:1X04
- added JP4, JP5: (no value), pinhead:1X03
- added JP6: (no value), pinhead:1X02
- added R12: 5.1K, joyAnalog:0805
- added SW1: 324_SW, 3pos_slide_switch_centered:342_SWICH_FOOT
- R8: value 1K -> 5K
- moved R6 109.3 mm to (5.31, 2.24), turned to 180 degrees
- moved LED2 109.3 mm to (5.29, 4.48), turned to 90 degrees
- moved C2 102.0 mm to (29.8, 67.4), turned to 90 degrees
- moved SW3 98.5 mm to (30.7, 41.4), turned to 270 degrees
- moved C1 97.5 mm to (29.8, 62.9), turned to 270 degrees
- moved R5 87.0 mm to (26.1, 36.9), turned to 0 degrees
- moved C4 85.7 mm to (40.5, 48.9), turned to 180 degrees
- moved SW4 83.6 mm to (25.9, 41.4), turned to 270 degrees
- moved R1 83.2 mm to (32.8, 57.7)
- moved R2 81.1 mm to (43.1, 57.7)
- moved LED3 77.0 mm to (32.0, 13.7)
- moved R3 72.4 mm to (36.3, 13.7), turned to 180 degrees
- moved C27 30.3 mm to (51.1, 10.5), turned to 0 degrees
- moved C5 24.1 mm to (57.5, 9.53)
- moved C3 23.0 mm to (50.8, 13.5)
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Connections:
- new net N$17: JP1.2, JP2.2, JP4.2
- new net N$19: F3.3, F3.4, J2.1, LED6.A
- new net N$21: IC3.12, JP1.4, JP7.3
- new net N$22: IC3.13, JP2.3, JP7.2
- new net N$23: IC3.14, JP2.4, JP7.1
- new net N$24: IC3.2, JP5.1
- new net N$25: J1.16, JP5.2
- new net N$26: IC3.3, J10.1, JP6.1, R12.1, SW1.P$2, SW1.P$3
- new net N$27: IC3.6, JP8.4
- new net N$28: J1.8, J9.1, LED3.A
- new net N$30: IC3.7, JP8.3
- new net N$32: IC3.10, JP8.2
- net +3V3: now also R12.2; no longer LED2.A, LED3.A
- net GND: now also J10.2, J2.2, J3.2, J4.2, J6.2, J7.2, J8.2, J9.2, JP1.1, JP2.1, JP5.3, JP6.2, JP8.1, R3.1, SW1.P$1, SW1.P$4; no longer J5.1, J5.2
- net N$11: no longer J4.2
- net N$14: now also IC3.11, JP1.3, JP7.4; no longer F2.1, F2.2, J6.1, J6.2, LED5.A
- net N$15: now also JP4.1; no longer J7.2
- net N$16: now also F2.1, F2.2, J6.1, JP4.3, LED5.A; no longer F3.3, F3.4, J2.1, J2.2, LED6.A
- net N$2: no longer J3.2
- net VCC: now also J8.1, LED2.A
Routing:
- net N$2: track 0.00 -> 116.7 mm
- net N$12: track 0.00 -> 112.8 mm
- net VCC: track 0.00 -> 109.0 mm
- net N$10: track 0.00 -> 82.2 mm
- net N$13: track 0.00 -> 64.0 mm
- net N$28: track 0.00 -> 56.7 mm
- net N$26: track 0.00 -> 48.7 mm
- net N$11: track 0.00 -> 48.2 mm
- net N$15: track 0.00 -> 43.2 mm
- net N$14: track 0.00 -> 41.4 mm
- net N$21: track 0.00 -> 40.3 mm
- net N$6: track 0.00 -> 36.7 mm
- net N$16: track 0.00 -> 34.0 mm
- net +3V3: track 0.00 -> 31.3 mm, vias 0 -> 6
- net N$22: track 0.00 -> 29.7 mm
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Other:
- board text added: "-12V"
- board text added: "12V"
- board text added: "5V"
- board text added: "5VSB"
- board text added: "DFU"
- board text added: "FUSE 3A MAX"
- board text added: "GND"
- board text added: "ON"
- board text added: "PWM"
- board text added: "PWR HEADER"
- board text added: "PWR OK"
- board text added: "PWR SW"
- board text added: "RST"
- board text added: "SEN"
- board text added: "SOFT PWR"
- board text added: "VFAN"
- board text removed: "CLK"
- board text removed: "DIO"
- board text removed: "RX"
- board text removed: "TX"

Commit message: working on PCB
Parts:
- added JP9: (no value), pinhead:1X03
- added R11: 1K, SparkFun-Passives:0805
- moved LED1 2.98 mm to (85.2, 17.0), turned to 90 degrees
- moved R7 2.92 mm to (85.2, 23.7), turned to 180 degrees
- moved LED4 1.90 mm to (85.2, 26.5), turned to 90 degrees
- moved R4 1.64 mm to (85.2, 14.9), turned to 180 degrees
Connections:
- new net N$34: JP9.2, R11.2
- net GND: now also J2.1, J3.1, J4.1, J6.1, J7.1, R11.1; no longer J2.2, J3.2, J4.2, J6.2, J7.2
- net N$11: now also J4.2; no longer J4.1
- net N$15: now also J7.2, JP9.1; no longer J7.1
- net N$16: now also J6.2; no longer J6.1
- net N$19: now also J2.2, JP9.3; no longer J2.1
- net N$2: now also J3.2; no longer J3.1
Routing:
- net N$15: track 43.2 -> 61.8 mm
- net N$19: track 22.5 -> 30.5 mm
- net N$34: track 0.00 -> 3.37 mm
- net N$2: track 116.7 -> 114.2 mm
- net N$16: track 34.0 -> 32.5 mm
- net N$17: track 24.0 -> 25.2 mm
- net N$11: track 48.2 -> 47.2 mm
- net N$8: track 2.09 -> 2.86 mm
Other:
- board text added: "ATX CONTROL BOARD dekuNukem July 2022 PT0"

Commit message: working on PCB
Parts:
- added R13: (no value), SparkFun-Retired:TRIM_POT_PTH
- moved JP6 7.00 mm to (44.1, 22.6)
- moved JP7 4.64 mm to (49.3, 48.8), turned to 0 degrees
- moved JP8 0.80 mm to (49.3, 41.1)
Connections:
- net +3V3: now also R13.1
- net GND: now also R13.3
- net N$27: now also R13.2
Routing:
- net N$27: track 17.8 -> 26.3 mm
- net GND: track 9.75 -> 4.40 mm
- net N$26: track 48.7 -> 44.3 mm
- net N$21: track 40.3 -> 42.9 mm
- net N$14: track 41.4 -> 43.7 mm
- net N$22: track 29.7 -> 31.9 mm
- net N$30: track 13.4 -> 15.3 mm
- net N$32: track 7.84 -> 9.15 mm
- net N$23: track 28.8 -> 29.7 mm
- net N$10: track 82.2 -> 81.6 mm
Other:
- board text added: "PA0"
- board text added: "PA1"
- board text added: "PA4"
- board text added: "PA5"
- board text added: "PA6"
- board text added: "PA7"
- board text added: "PB1"
- board text added: "PWR ON"

Commit message: pcb done sent to fab
Parts:
- moved R1 0.77 mm to (33.5, 57.8)
- moved JP4 0.76 mm to (69.6, 58.2)
- moved R5 0.64 mm to (25.4, 36.9)
- moved SW3 0.64 mm to (30.1, 41.4)
- moved SW4 0.64 mm to (25.3, 41.4)
- moved JP6 0.40 mm to (43.9, 22.2)
- moved R2 0.28 mm to (43.3, 57.8)
Routing:
- net GND: track 4.40 -> 31.8 mm
- net N$6: track 36.7 -> 35.8 mm
- net VCC: track 108.9 -> 109.7 mm
- net N$31: track 7.14 -> 6.32 mm
- net N$17: track 25.2 -> 26.0 mm
- net N$16: track 32.5 -> 31.7 mm
- net N$15: track 61.8 -> 61.0 mm
- net N$14: track 43.7 -> 44.4 mm
- net BUTTON2: track 18.5 -> 19.2 mm
- net BUTTON1: track 10.8 -> 11.4 mm
- net N$26: track 44.3 -> 43.7 mm
