File: pcb/atx_power_control.sch (EAGLE design)
At the start: 25 parts, among them IC3 STM32F042F4, SW3 324_SW, SW4 324_SW, U2 USBC_16P, U4 XC6206_DEV

Commit message: working on PCB
Parts:
- removed JP1: (no value), pmm:PINHEAD_PINHD-2X4
- removed R7: 1K, SparkFun-Passives:RESISTOR0805-RES
- removed TP1, TP2, TP3, TP4, TP5: TPSQTP10SQ, testpad:TPSQTP10SQ
- removed U4: XC6206_DEV, 3pos_slide_switch:XC6206_DEV
- added C3: 2.2uF, clock:CAP0805
- added C5: 1uF, clock:CAP0805
- added D3: (no value), adafruit:DIODE_SOD-123FL
- added F1, F2, F3: FUSEX20MM, atx_power_control:FUSEX20MM
- added IC2: REG1117, clock:REG1117
- added IC4: MY_7905DT, atx_power_control:MY_7905DT
- added J1: ATX24RH, SparkFun-Connectors:ATX24RH
- added J2, J3, J4, J5, J6, J7: (no value), SparkFun-Connectors:CONN_023.5MM
- added U$1, U$10, U$2, U$3: M3_MOUNTING_HOLE, a:M3_MOUNTING_HOLE
Connections:
- removed net +5V: C1.2, U2.VBUS, U4.IN
- removed net N$15: IC3.PA4, TP5.TP
- removed net SCL: IC3.PF1/OSC_OUT, JP1.5, JP1.6
- new net VCC: C1.2, D3.C, IC2.VIN, J1.5V_STDBY
- net +3V3: now also IC2.VOUT; no longer R7.2, U4.OUT
- net GND: now also C3.1, C5.1, IC2.GND, IC4.GND, J1.GND@0, J1.GND@1, J1.GND@2, J1.GND@3, J1.GND@4, J1.GND@5, J1.GND@6, J1.GND@7, J5.1, J5.2; no longer JP1.7, JP1.8, U4.GND
- net N$10: now also D3.A, U2.VBUS; no longer JP1.1, JP1.2, R7.1
- net N$11: now also C5.2, IC4.VO, J4.1, J4.2; no longer IC3.PA7, TP4.TP
- net N$12: now also J1.3.3V@0, J1.3.3V@1, J1.3.3V@2, J1.3.3V@3; no longer IC3.PA6, TP3.TP
- net N$13: now also F2.2, J1.12V@0, J1.12V@1; no longer IC3.PA5, TP2.TP
- net N$14: now also F2.1, J6.1, J6.2; no longer IC3.PB1, TP1.TP
- net N$2: now also C3.2, IC4.VI, J1.-12V, J3.1, J3.2; no longer IC3.PF0/OSC_IN, JP1.3, JP1.4
