File: pcb/atx_power_control.sch (EAGLE design)
At the start: 36 parts, among them IC2 REG1117, IC3 STM32F042F4, IC4 MY_7905DT, J1 ATX24RH, SW3 324_SW, SW4 324_SW, U2 USBC_16P

Commit message: working on PCB
Parts:
- removed D3: (no value), adafruit:DIODE_SOD-123FL
- added C27: 47uF, clock:C-USC1210
- added IC1: (no value), linear:7905T
- added LED4, LED5, LED6, LED7: (no value), adafruit:LEDCHIP-LED0805
- added R10, R8, R9: 1K, SparkFun-Passives:RESISTOR0805-RES
- added R7: 5K, SparkFun-Passives:RESISTOR0805-RES
Connections:
- new net N$15: F1.2, J7.1, J7.2, LED7.A
- new net N$16: F3.2, J2.1, J2.2, LED6.A
- new net N$18: LED6.C, R9.2
- new net N$20: LED7.C, R10.2
- net +3V3: no longer LED1.A
- net GND: now also C27.2, IC1.GND, LED1.A, LED4.A, R10.1, R8.1, R9.1
- net N$10: now also F1.1, J1.5V@0, J1.5V@1, J1.5V@2, J1.5V@3, J1.5V@4; no longer D3.A, U2.VBUS
- net N$11: now also IC1.VO, R4.1
- net N$12: now also F3.1
- net N$14: now also LED5.A
- net N$2: now also C27.1, IC1.VI, R7.1
- net N$8: now also LED4.C, R7.2; no longer IC3.PA0, R4.1
- net N$9: now also LED5.C, R8.2; no longer IC3.PA1, R3.1
- net VCC: now also U2.VBUS; no longer D3.C
Other:
- moved on the sheet: F1, F3, J2, J7, LED1, R4

Commit message: working on PCB
Parts:
- removed J5: (no value), SparkFun-Connectors:CONN_023.5MM
- added J10, J8, J9: (no value), SparkFun-Connectors:CONN_023.5MM
- added JP1, JP2, JP7, JP8: (no value), pinhead:PINHD-1X4
- added JP4, JP5: (no value), pinhead:PINHD-1X3
- added JP6: (no value), pinhead:PINHD-1X2
- added R12: 5.1K, joyAnalog:RESISTOR0805-RES
- added SW1: 324_SW, 3pos_slide_switch_centered:324_SW
- R8: value 1K -> 5K
Connections:
- new net N$17: JP1.2, JP2.2, JP4.2
- new net N$19: F3.2, J2.1, LED6.A
- new net N$21: IC3.PA6, JP1.4, JP7.3
- new net N$22: IC3.PA7, JP2.3, JP7.2
- new net N$23: IC3.PB1, JP2.4, JP7.1
- new net N$24: IC3.PF0/OSC_IN, JP5.1
- new net N$25: J1.PS_ON, JP5.2
- new net N$26: IC3.PF1/OSC_OUT, J10.1, JP6.1, R12.1, SW1.2, SW1.3
- new net N$27: IC3.PA0, JP8.4
- new net N$28: J1.PWR_OK, J9.1, LED3.A
- new net N$30: IC3.PA1, JP8.3
- new net N$32: IC3.PA4, JP8.2
- net +3V3: now also R12.2; no longer LED2.A, LED3.A
- net GND: now also J10.2, J2.2, J3.2, J4.2, J6.2, J7.2, J8.2, J9.2, JP1.1, JP2.1, JP5.3, JP6.2, JP8.1, R3.1, SW1.1, SW1.4; no longer J5.1, J5.2
- net N$11: no longer J4.2
- net N$14: now also IC3.PA5, JP1.3, JP7.4; no longer F2.1, J6.1, J6.2, LED5.A
- net N$15: now also JP4.1; no longer J7.2
- net N$16: now also F2.1, J6.1, JP4.3, LED5.A; no longer F3.2, J2.1, J2.2, LED6.A
- net N$2: no longer J3.2
- net VCC: now also J8.1, LED2.A
Other:
- moved on the sheet: LED2, LED3, R3, R6

Commit message: working on PCB
Parts:
- added JP9: (no value), pinhead:PINHD-1X3
- added R11: 1K, SparkFun-Passives:RESISTOR0805-RES
Connections:
- new net N$34: JP9.2, R11.2
- net GND: now also J2.1, J3.1, J4.1, J6.1, J7.1, R11.1; no longer J2.2, J3.2, J4.2, J6.2, J7.2
- net N$11: now also J4.2; no longer J4.1
- net N$15: now also J7.2, JP9.1; no longer J7.1
- net N$16: now also J6.2; no longer J6.1
- net N$19: now also J2.2, JP9.3; no longer J2.1
- net N$2: now also J3.2; no longer J3.1

Commit message: working on PCB
Parts:
- added R13: (no value), SparkFun-Retired:TRIMPOTPTH
Connections:
- net +3V3: now also R13.CCW
- net GND: now also R13.CW
- net N$27: now also R13.WIPER
Changed lines of the file:
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@@
 <part name="R11" library="SparkFun-Passives" deviceset="RESISTOR" device="0805-RES" value="1K"/>
 <part name="GND34" library="backplane" deviceset="GND" device=""/>
+<part name="R13" library="SparkFun-Retired" deviceset="TRIMPOT" device="PTH"/>
+<part name="+3V4" library="supply1" library_urn="urn:adsk.eagle:library:371" deviceset="+3V3" device=""/>
+<part name="GND35" library="supply1" deviceset="GND" device=""/>
 </parts>
 <sheets>
@@
 <instance part="GND34" gate="1" x="317.5" y="76.2" smashed="yes" rot="R180">
 <attribute name="VALUE" x="320.04" y="78.74" size="1.778" layer="96" rot="R180"/>
+</instance>
+<instance part="R13" gate="R?" x="-88.9" y="25.4" smashed="yes">
+<attribute name="NAME" x="-90.17" y="21.8186" size="1.778" layer="95"/>
+<attribute name="VALUE" x="-92.71" y="22.098" size="1.778" layer="96"/>
+</instance>
+<instance part="+3V4" gate="G$1" x="-99.06" y="27.94" smashed="yes" rot="MR0">
+<attribute name="VALUE" x="-96.52" y="22.86" size="1.778" layer="96" rot="MR90"/>
+</instance>
+<instance part="GND35" gate="1" x="-81.28" y="22.86" smashed="yes" rot="MR0">
+<attribute name="VALUE" x="-78.74" y="20.32" size="1.778" layer="96" rot="MR0"/>
 </instance>
 </instances>
@@
 <pinref part="GND34" gate="1" pin="GND"/>
 </segment>
+<segment>
+<pinref part="R13" gate="R?" pin="CW"/>
+<pinref part="GND35" gate="1" pin="GND"/>
+<wire x1="-83.82" y1="25.4" x2="-81.28" y2="25.4" width="0.1524" layer="91"/>
+</segment>
 </net>
 <net name="+3V3" class="0">
@@
 <pinref part="R12" gate="G$1" pin="2"/>
 <pinref part="+3V3" gate="G$1" pin="+3V3"/>
+</segment>
+<segment>
+<pinref part="+3V4" gate="G$1" pin="+3V3"/>
+<pinref part="R13" gate="R?" pin="CCW"/>
+<wire x1="-99.06" y1="25.4" x2="-93.98" y2="25.4" width="0.1524" layer="91"/>
 </segment>
 </net>
@@
 <pinref part="JP8" gate="A" pin="4"/>
 <wire x1="-17.78" y1="40.64" x2="-60.96" y2="40.64" width="0.1524" layer="91"/>
-</segment>
-</net>
+<pinref part="R13" gate="R?" pin="WIPER"/>
+<wire x1="-88.9" y1="30.48" x2="-88.9" y2="40.64" width="0.1524" layer="91"/>
+<wire x1="-88.9" y1="40.64" x2="-60.96" y2="40.64" width="0.1524" layer="91"/>
+<junction x="-60.96" y="40.64"/>
+</segment>
+</net>
