File: pcb/nomcu.sch (EAGLE design)
At the start: 35 parts, among them IC4 MY_7905DT, J1 ATX24RH

Commit message: working on daughterboard
Parts:
- removed JP16: (no value), appleii:4PIN_FAN
- added JP2: (no value), pinhead:PINHD-1X4
- JP3: device pinhead:PINHD-2X3 -> pinhead:PINHD-2X4
Connections:
- removed net N$2: JP16.4_PWM, JP8.4_PWM
- net F12V: no longer JP16.2_VCC
- net GND: no longer JP16.1_GND
Changed lines of the file:
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@@
 <part name="GND22" library="supply1" deviceset="GND" device=""/>
 <part name="JP8" library="appleii" deviceset="4PIN_FAN" device=""/>
-<part name="JP16" library="appleii" deviceset="4PIN_FAN" device=""/>
-<part name="GND23" library="supply1" deviceset="GND" device=""/>
 <part name="GND26" library="supply1" deviceset="GND" device=""/>
 <part name="J4" library="SparkFun-Connectors" deviceset="USB_C" device="16PIN"/>
-<part name="JP3" library="pinhead" library_urn="urn:adsk.eagle:library:325" deviceset="PINHD-2X3" device="" package3d_urn="urn:adsk.eagle:package:22462/2"/>
+<part name="JP3" library="pinhead" library_urn="urn:adsk.eagle:library:325" deviceset="PINHD-2X4" device="" package3d_urn="urn:adsk.eagle:package:22461/2"/>
+<part name="JP2" library="pinhead" library_urn="urn:adsk.eagle:library:325" deviceset="PINHD-1X4" device="" package3d_urn="urn:adsk.eagle:package:22407/2"/>
 </parts>
 <sheets>
@@
 </instance>
 <instance part="JP8" gate="A" x="251.46" y="-93.98" smashed="yes" rot="R180"/>
-<instance part="JP16" gate="A" x="195.58" y="-93.98" smashed="yes" rot="R180"/>
-<instance part="GND23" gate="1" x="213.36" y="-104.14" smashed="yes" rot="MR0">
-<attribute name="VALUE" x="215.9" y="-106.68" size="1.778" layer="96" rot="MR0"/>
-</instance>
 <instance part="GND26" gate="1" x="269.24" y="-104.14" smashed="yes" rot="MR0">
 <attribute name="VALUE" x="271.78" y="-106.68" size="1.778" layer="96" rot="MR0"/>
@@
 <attribute name="NAME" x="140.97" y="28.575" size="1.778" layer="95"/>
 <attribute name="VALUE" x="140.97" y="15.24" size="1.778" layer="96"/>
+</instance>
+<instance part="JP2" gate="A" x="215.9" y="-93.98" smashed="yes">
+<attribute name="NAME" x="209.55" y="-85.725" size="1.778" layer="95"/>
+<attribute name="VALUE" x="209.55" y="-101.6" size="1.778" layer="96"/>
 </instance>
 </instances>
@@
 <pinref part="GND22" gate="1" pin="GND"/>
 <wire x1="370.84" y1="-43.18" x2="408.94" y2="-43.18" width="0.1524" layer="91"/>
-</segment>
-<segment>
-<pinref part="JP16" gate="A" pin="1_GND"/>
-<pinref part="GND23" gate="1" pin="GND"/>
-<wire x1="208.28" y1="-101.6" x2="213.36" y2="-101.6" width="0.1524" layer="91"/>
 </segment>
 <segment>
@@
 <wire x1="383.54" y1="-27.94" x2="370.84" y2="-27.94" width="0.1524" layer="91"/>
 <junction x="383.54" y="12.7"/>
-<pinref part="JP16" gate="A" pin="2_VCC"/>
 <wire x1="304.8" y1="-96.52" x2="264.16" y2="-96.52" width="0.1524" layer="91"/>
 <pinref part="JP8" gate="A" pin="2_VCC"/>
-<wire x1="264.16" y1="-96.52" x2="208.28" y2="-96.52" width="0.1524" layer="91"/>
-<junction x="264.16" y="-96.52"/>
 <pinref part="U$4" gate="G$1" pin="P$5"/>
 <wire x1="335.28" y1="66.04" x2="386.08" y2="66.04" width="0.1524" layer="91"/>
@@
 </segment>
 </net>
-<net name="N$2" class="0">
-<segment>
-<pinref part="JP8" gate="A" pin="4_PWM"/>
-<pinref part="JP16" gate="A" pin="4_PWM"/>
-<wire x1="208.28" y1="-86.36" x2="264.16" y2="-86.36" width="0.1524" layer="91"/>
-</segment>
-</net>

Commit message: working on new version
Parts:
- removed JP5: (no value), atx_power_control:PINHD-1X3:1
- added U$11, U$6: M3_MOUNTING_HOLE, a:M3_MOUNTING_HOLE
- JP2: device pinhead:PINHD-1X4 -> pinhead:PINHD-1X2
- U$9: value WAGO257-7 -> DG2204R-5.0; device atx4vc:WAGO257-7 -> atx4vc:DG2204R-5.0
Connections:
- net -12V: now also U$9.P$7; no longer U$9.P$1
- net -5V: now also U$9.P$6; no longer U$9.P$2
- net F12V: now also U$9.P$3; no longer U$9.P$7
- net F3V3: now also U$9.P$5; no longer U$9.P$3
- net F5V: now also U$9.P$4; no longer U$9.P$5
- net GND: now also JP2.1, U$9.P$1, U$9.P$2; no longer JP5.3, U$9.P$4, U$9.P$6
- net N$15: now also JP2.2; no longer JP5.2
Changed lines of the file:
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@@
 <part name="R10" library="atx_power_control" deviceset="RESISTOR" device="0805-RES" value="5K1"/>
 <part name="GND21" library="backplane" deviceset="GND" device=""/>
-<part name="JP5" library="atx_power_control" deviceset="PINHD-1X3*?:1" device=""/>
 <part name="GND24" library="supply1" deviceset="GND" device=""/>
 <part name="GND32" library="supply1" deviceset="GND" device=""/>
@@
 <part name="GND37" library="backplane" deviceset="GND" device=""/>
 <part name="R22" library="atx_power_control" deviceset="RESISTOR" device="0805-RES" value="5K1"/>
-<part name="U$9" library="atx4vc" deviceset="WAGO257-7" device=""/>
+<part name="U$9" library="atx4vc" deviceset="DG2204R-5.0" device=""/>
 <part name="GND14" library="supply1" deviceset="GND" device=""/>
-<part name="GND22" library="supply1" deviceset="GND" device=""/>
 <part name="JP8" library="appleii" deviceset="4PIN_FAN" device=""/>
 <part name="GND26" library="supply1" deviceset="GND" device=""/>
 <part name="J4" library="SparkFun-Connectors" deviceset="USB_C" device="16PIN"/>
 <part name="JP3" library="pinhead" library_urn="urn:adsk.eagle:library:325" deviceset="PINHD-2X4" device="" package3d_urn="urn:adsk.eagle:package:22461/2"/>
-<part name="JP2" library="pinhead" library_urn="urn:adsk.eagle:library:325" deviceset="PINHD-1X4" device="" package3d_urn="urn:adsk.eagle:package:22407/2"/>
+<part name="U$6" library="a" deviceset="M3_MOUNTING_HOLE" device=""/>
+<part name="U$11" library="a" deviceset="M3_MOUNTING_HOLE" device=""/>
+<part name="JP2" library="pinhead" library_urn="urn:adsk.eagle:library:325" deviceset="PINHD-1X2" device="" package3d_urn="urn:adsk.eagle:package:22435/2"/>
 </parts>
 <sheets>
@@
 <attribute name="VALUE" x="447.04" y="38.1" size="1.778" layer="96"/>
 </instance>
-<instance part="JP5" gate="A" x="185.42" y="-33.02" smashed="yes">
-<attribute name="NAME" x="179.07" y="-27.305" size="1.778" layer="95"/>
-<attribute name="VALUE" x="179.07" y="-40.64" size="1.778" layer="96"/>
-</instance>
 <instance part="GND24" gate="1" x="172.72" y="-38.1" smashed="yes" rot="MR0">
 <attribute name="VALUE" x="175.26" y="-40.64" size="1.778" layer="96" rot="MR0"/>
@@
 <attribute name="VALUE" x="309.118" y="77.47" size="1.778" layer="96" rot="R270"/>
 </instance>
-<instance part="U$9" gate="G$1" x="360.68" y="-58.42" smashed="yes" rot="R180"/>
-<instance part="GND14" gate="1" x="408.94" y="-35.56" smashed="yes" rot="MR0">
-<attribute name="VALUE" x="411.48" y="-38.1" size="1.778" layer="96" rot="MR0"/>
-</instance>
-<instance part="GND22" gate="1" x="408.94" y="-45.72" smashed="yes" rot="MR0">
-<attribute name="VALUE" x="411.48" y="-48.26" size="1.778" layer="96" rot="MR0"/>
+<instance part="U$9" gate="G$1" x="370.84" y="-27.94" smashed="yes" rot="MR0"/>
+<instance part="GND14" gate="1" x="355.6" y="-35.56" smashed="yes" rot="MR0">
+<attribute name="VALUE" x="358.14" y="-38.1" size="1.778" layer="96" rot="MR0"/>
 </instance>
 <instance part="JP8" gate="A" x="251.46" y="-93.98" smashed="yes" rot="R180"/>
@@
 <attribute name="VALUE" x="140.97" y="15.24" size="1.778" layer="96"/>
 </instance>
-<instance part="JP2" gate="A" x="215.9" y="-93.98" smashed="yes">
-<attribute name="NAME" x="209.55" y="-85.725" size="1.778" layer="95"/>
-<attribute name="VALUE" x="209.55" y="-101.6" size="1.778" layer="96"/>
+<instance part="U$6" gate="G$1" x="223.52" y="91.44" smashed="yes"/>
+<instance part="U$11" gate="G$1" x="215.9" y="109.22" smashed="yes"/>
+<instance part="JP2" gate="G$1" x="160.02" y="-33.02" smashed="yes" rot="R180">
+<attribute name="NAME" x="166.37" y="-38.735" size="1.778" layer="95" rot="R180"/>
+<attribute name="VALUE" x="166.37" y="-27.94" size="1.778" layer="96" rot="R180"/>
 </instance>
 </instances>
@@
 </segment>
 <segment>
-<pinref part="JP5" gate="A" pin="3"/>
-<pinref part="GND24" gate="1" pin="GND"/>
-<wire x1="182.88" y1="-35.56" x2="172.72" y2="-35.56" width="0.1524" layer="91"/>
-</segment>
-<segment>
 <pinref part="R3" gate="G$1" pin="1"/>
 <pinref part="GND32" gate="1" pin="GND"/>
@@
 <pinref part="GND33" gate="1" pin="GND"/>
 <wire x1="317.5" y1="144.78" x2="317.5" y2="106.68" width="0.1524" layer="91"/>
-</segment>
-<segment>
-<pinref part="U$9" gate="G$1" pin="P$6"/>
-<pinref part="GND14" gate="1" pin="GND"/>
-<wire x1="370.84" y1="-33.02" x2="408.94" y2="-33.02" width="0.1524" layer="91"/>
-</segment>
-<segment>
-<pinref part="U$9" gate="G$1" pin="P$4"/>
-<pinref part="GND22" gate="1" pin="GND"/>
-<wire x1="370.84" y1="-43.18" x2="408.94" y2="-43.18" width="0.1524" layer="91"/>
 </segment>
 <segment>
@@
 <wire x1="386.08" y1="60.96" x2="406.4" y2="60.96" width="0.1524" layer="91"/>
 <junction x="406.4" y="60.96"/>
+</segment>
+<segment>
+<pinref part="GND14" gate="1" pin="GND"/>
+<pinref part="U$9" gate="G$1" pin="P$2"/>
+<wire x1="355.6" y1="-33.02" x2="381" y2="-33.02" width="0.1524" layer="91"/>
+<pinref part="U$9" gate="G$1" pin="P$1"/>
+<wire x1="355.6" y1="-33.02" x2="355.6" y2="-27.94" width="0.1524" layer="91"/>
+<wire x1="355.6" y1="-27.94" x2="381" y2="-27.94" width="0.1524" layer="91"/>
+<junction x="355.6" y="-33.02"/>
+</segment>
+<segment>
+<pinref part="GND24" gate="1" pin="GND"/>
+<pinref part="JP2" gate="G$1" pin="1"/>
+<wire x1="172.72" y1="-35.56" x2="162.56" y2="-35.56" width="0.1524" layer="91"/>
 </segment>
 </net>
@@
 <pinref part="R7" gate="G$1" pin="1"/>
 <wire x1="408.94" y1="0" x2="421.64" y2="0" width="0.1524" layer="91"/>
-<pinref part="U$9" gate="G$1" pin="P$1"/>
 <wire x1="403.86" y1="-2.54" x2="403.86" y2="-58.42" width="0.1524" layer="91"/>
-<wire x1="403.86" y1="-58.42" x2="370.84" y2="-58.42" width="0.1524" layer="91"/>
 <junction x="403.86" y="-2.54"/>
+<wire x1="403.86" y1="-58.42" x2="381" y2="-58.42" width="0.1524" layer="91"/>
+<pinref part="U$9" gate="G$1" pin="P$7"/>
 </segment>
 </net>
@@
 <wire x1="337.82" y1="73.66" x2="337.82" y2="-15.24" width="0.1524" layer="91"/>
 <junction x="337.82" y="-15.24"/>
-<pinref part="U$9" gate="G$1" pin="P$2"/>
 <wire x1="398.78" y1="-15.24" x2="398.78" y2="-53.34" width="0.1524" layer="91"/>
-<wire x1="398.78" y1="-53.34" x2="370.84" y2="-53.34" width="0.1524" layer="91"/>
 <junction x="398.78" y="-15.24"/>
+<pinref part="U$9" gate="G$1" pin="P$6"/>
+<wire x1="398.78" y1="-53.34" x2="381" y2="-53.34" width="0.1524" layer="91"/>
 </segment>
 </net>
@@
 <pinref part="R22" gate="G$1" pin="2"/>
 <wire x1="314.96" y1="68.58" x2="312.42" y2="68.58" width="0.1524" layer="91"/>
-<pinref part="U$9" gate="G$1" pin="P$5"/>
-<wire x1="388.62" y1="40.64" x2="388.62" y2="-38.1" width="0.1524" layer="91"/>
-<wire x1="388.62" y1="-38.1" x2="370.84" y2="-38.1" width="0.1524" layer="91"/>
+<wire x1="388.62" y1="40.64" x2="388.62" y2="-43.18" width="0.1524" layer="91"/>
 <junction x="388.62" y="40.64"/>
 <pinref part="J4" gate="J1" pin="VBUS"/>
 <pinref part="U$4" gate="G$1" pin="P$4"/>
 <wire x1="332.74" y1="68.58" x2="386.08" y2="68.58" width="0.1524" layer="91"/>
+<pinref part="U$9" gate="G$1" pin="P$4"/>
+<wire x1="388.62" y1="-43.18" x2="381" y2="-43.18" width="0.1524" layer="91"/>
 </segment>
 </net>
@@
 <wire x1="335.28" y1="66.04" x2="335.28" y2="5.08" width="0.1524" layer="91"/>
 <junction x="335.28" y="5.08"/>
-<pinref part="U$9" gate="G$1" pin="P$7"/>
-<wire x1="383.54" y1="12.7" x2="383.54" y2="-27.94" width="0.1524" layer="91"/>
-<wire x1="383.54" y1="-27.94" x2="370.84" y2="-27.94" width="0.1524" layer="91"/>
+<wire x1="383.54" y1="12.7" x2="383.54" y2="-38.1" width="0.1524" layer="91"/>
 <junction x="383.54" y="12.7"/>
 <wire x1="304.8" y1="-96.52" x2="264.16" y2="-96.52" width="0.1524" layer="91"/>
@@
 <pinref part="U$4" gate="G$1" pin="P$5"/>
 <wire x1="335.28" y1="66.04" x2="386.08" y2="66.04" width="0.1524" layer="91"/>
+<pinref part="U$9" gate="G$1" pin="P$3"/>
+<wire x1="383.54" y1="-38.1" x2="381" y2="-38.1" width="0.1524" layer="91"/>
 </segment>
 </net>
@@
 <wire x1="330.2" y1="71.12" x2="330.2" y2="22.86" width="0.1524" layer="91"/>
 <junction x="330.2" y="22.86"/>
-<pinref part="U$9" gate="G$1" pin="P$3"/>
 <wire x1="393.7" y1="22.86" x2="393.7" y2="-48.26" width="0.1524" layer="91"/>
-<wire x1="393.7" y1="-48.26" x2="370.84" y2="-48.26" width="0.1524" layer="91"/>
 <junction x="393.7" y="22.86"/>
+<pinref part="U$9" gate="G$1" pin="P$5"/>
+<wire x1="393.7" y1="-48.26" x2="381" y2="-48.26" width="0.1524" layer="91"/>
 </segment>
 </net>
@@
 <net name="N$15" class="0">
 <segment>
-<pinref part="JP5" gate="A" pin="2"/>
 <pinref part="J1" gate="G$1" pin="PS_ON"/>
 <wire x1="259.08" y1="-7.62" x2="248.92" y2="-7.62" width="0.1524" layer="91"/>
 <wire x1="259.08" y1="-33.02" x2="259.08" y2="-7.62" width="0.1524" layer="91"/>
-<wire x1="259.08" y1="-33.02" x2="182.88" y2="-33.02" width="0.1524" layer="91"/>
-</segment>
-</net>
+<wire x1="259.08" y1="-33.02" x2="162.56" y2="-33.02" width="0.1524" layer="91"/>
+<pinref part="JP2" gate="G$1" pin="2"/>
+</segment>
+</net>

Commit message: working on new version
Parts:
- added JP4: (no value), pinhead:PINHD-2X2
- added U$12: PINHD1X4, adafruit_changed:PINHD1X4
- J1: device SparkFun-Connectors:ATX24RH -> nomcu:ATX24RH
- JP3: device pinhead:PINHD-2X4 -> pinhead:PINHD-2X3
Connections:
- new net N$3: JP3.3, JP8.4_PWM
- new net N$4: J4.D+, JP4.2
- new net N$6: J4.D-, JP4.4
- new net N$7: JP3.4, JP4.1, JP4.3, U$12.2
- net F5V: now also U$12.1
- net GND: now also JP3.2, U$12.4
- net N$11: now also JP3.5
- net N$15: now also JP3.6
- net VCC: now also JP3.1
Other:
- moved on the sheet: JP2
Changed lines of the file:
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@@
 <part name="U$2" library="a" deviceset="M3_MOUNTING_HOLE" device=""/>
 <part name="U$3" library="a" deviceset="M3_MOUNTING_HOLE" device=""/>
-<part name="J1" library="SparkFun-Connectors" deviceset="ATX24" device="RH"/>
+<part name="J1" library="nomcu" deviceset="ATX24" device="RH"/>
 <part name="GND2" library="supply1" deviceset="GND" device=""/>
 <part name="SUPPLY5" library="supply2" library_urn="urn:adsk.eagle:library:372" deviceset="VCC" device=""/>
@@
 <part name="GND26" library="supply1" deviceset="GND" device=""/>
 <part name="J4" library="SparkFun-Connectors" deviceset="USB_C" device="16PIN"/>
-<part name="JP3" library="pinhead" library_urn="urn:adsk.eagle:library:325" deviceset="PINHD-2X4" device="" package3d_urn="urn:adsk.eagle:package:22461/2"/>
+<part name="JP3" library="pinhead" library_urn="urn:adsk.eagle:library:325" deviceset="PINHD-2X3" device="" package3d_urn="urn:adsk.eagle:package:22462/2"/>
 <part name="U$6" library="a" deviceset="M3_MOUNTING_HOLE" device=""/>
 <part name="U$11" library="a" deviceset="M3_MOUNTING_HOLE" device=""/>
 <part name="JP2" library="pinhead" library_urn="urn:adsk.eagle:library:325" deviceset="PINHD-1X2" device="" package3d_urn="urn:adsk.eagle:package:22435/2"/>
+<part name="SUPPLY1" library="supply2" library_urn="urn:adsk.eagle:library:372" deviceset="VCC" device=""/>
+<part name="GND1" library="supply1" deviceset="GND" device=""/>
+<part name="GND3" library="backplane" deviceset="GND" device=""/>
+<part name="U$12" library="adafruit_changed" deviceset="PINHD1X4" device=""/>
+<part name="JP4" library="pinhead" library_urn="urn:adsk.eagle:library:325" deviceset="PINHD-2X2" device="" package3d_urn="urn:adsk.eagle:package:22455/2"/>
 </parts>
 <sheets>
@@
 <attribute name="VALUE" x="447.04" y="38.1" size="1.778" layer="96"/>
 </instance>
-<instance part="GND24" gate="1" x="172.72" y="-38.1" smashed="yes" rot="MR0">
-<attribute name="VALUE" x="175.26" y="-40.64" size="1.778" layer="96" rot="MR0"/>
+<instance part="GND24" gate="1" x="241.3" y="-38.1" smashed="yes" rot="MR0">
+<attribute name="VALUE" x="243.84" y="-40.64" size="1.778" layer="96" rot="MR0"/>
 </instance>
 <instance part="GND32" gate="1" x="276.86" y="-45.72" smashed="yes" rot="MR0">
@@
 <attribute name="NAME" x="279.4" y="134.874" size="1.778" layer="95" font="vector"/>
 </instance>
-<instance part="JP3" gate="A" x="147.32" y="22.86" smashed="yes">
-<attribute name="NAME" x="140.97" y="28.575" size="1.778" layer="95"/>
-<attribute name="VALUE" x="140.97" y="15.24" size="1.778" layer="96"/>
+<instance part="JP3" gate="A" x="165.1" y="5.08" smashed="yes">
+<attribute name="VALUE" x="158.75" y="-2.54" size="1.778" layer="96"/>
 </instance>
 <instance part="U$6" gate="G$1" x="223.52" y="91.44" smashed="yes"/>
 <instance part="U$11" gate="G$1" x="215.9" y="109.22" smashed="yes"/>
-<instance part="JP2" gate="G$1" x="160.02" y="-33.02" smashed="yes" rot="R180">
-<attribute name="NAME" x="166.37" y="-38.735" size="1.778" layer="95" rot="R180"/>
-<attribute name="VALUE" x="166.37" y="-27.94" size="1.778" layer="96" rot="R180"/>
+<instance part="JP2" gate="G$1" x="228.6" y="-33.02" smashed="yes" rot="R180">
+<attribute name="NAME" x="234.95" y="-38.735" size="1.778" layer="95" rot="R180"/>
+<attribute name="VALUE" x="234.95" y="-27.94" size="1.778" layer="96" rot="R180"/>
+</instance>
+<instance part="SUPPLY1" gate="G$1" x="152.4" y="10.16" smashed="yes">
+<attribute name="VALUE" x="150.495" y="13.335" size="1.778" layer="96"/>
+</instance>
+<instance part="GND1" gate="1" x="182.88" y="5.08" smashed="yes" rot="MR0">
+<attribute name="VALUE" x="185.42" y="2.54" size="1.778" layer="96" rot="MR0"/>
+</instance>
+<instance part="GND3" gate="1" x="264.16" y="60.96" smashed="yes">
+<attribute name="VALUE" x="261.62" y="58.42" size="1.778" layer="96"/>
+</instance>
+<instance part="U$12" gate="1" x="248.92" y="58.42" smashed="yes" rot="R180">
+<attribute name="NAME" x="243.84" y="50.8" size="1.27" layer="95" font="vector"/>
+<attribute name="VALUE" x="248.92" y="68.58" size="1.27" layer="96" font="vector" rot="R180"/>
+</instance>
+<instance part="JP4" gate="A" x="251.46" y="127" smashed="yes">
+<attribute name="NAME" x="242.57" y="132.715" size="1.778" layer="95"/>
+<attribute name="VALUE" x="242.57" y="121.92" size="1.778" layer="96"/>
 </instance>
 </instances>
@@
 <pinref part="GND24" gate="1" pin="GND"/>
 <pinref part="JP2" gate="G$1" pin="1"/>
-<wire x1="172.72" y1="-35.56" x2="162.56" y2="-35.56" width="0.1524" layer="91"/>
+<wire x1="241.3" y1="-35.56" x2="231.14" y2="-35.56" width="0.1524" layer="91"/>
+</segment>
+<segment>
+<pinref part="GND1" gate="1" pin="GND"/>
+<pinref part="JP3" gate="A" pin="2"/>
+<wire x1="182.88" y1="7.62" x2="170.18" y2="7.62" width="0.1524" layer="91"/>
+</segment>
+<segment>
+<pinref part="U$12" gate="1" pin="4"/>
+<pinref part="GND3" gate="1" pin="GND"/>
+<wire x1="254" y1="63.5" x2="264.16" y2="63.5" width="0.1524" layer="91"/>
 </segment>
 </net>
@@
 <pinref part="SUPPLY6" gate="G$1" pin="VCC"/>
 <wire x1="220.98" y1="7.62" x2="205.74" y2="7.62" width="0.1524" layer="91"/>
+</segment>
+<segment>
+<pinref part="SUPPLY1" gate="G$1" pin="VCC"/>
+<pinref part="JP3" gate="A" pin="1"/>
+<wire x1="152.4" y1="7.62" x2="162.56" y2="7.62" width="0.1524" layer="91"/>
 </segment>
 </net>
@@
 <junction x="314.96" y="40.64"/>
 <pinref part="U$8" gate="G$1" pin="B0"/>
-<wire x1="307.34" y1="40.64" x2="297.434" y2="40.64" width="0.1524" layer="91"/>
 <wire x1="297.434" y1="40.64" x2="297.434" y2="39.37" width="0.1524" layer="91"/>
 <junction x="307.34" y="40.64"/>
@@
 <pinref part="U$9" gate="G$1" pin="P$4"/>
 <wire x1="388.62" y1="-43.18" x2="381" y2="-43.18" width="0.1524" layer="91"/>
+<wire x1="307.34" y1="40.64" x2="302.26" y2="40.64" width="0.1524" layer="91"/>
+<wire x1="302.26" y1="40.64" x2="297.434" y2="40.64" width="0.1524" layer="91"/>
+<wire x1="254" y1="55.88" x2="302.26" y2="55.88" width="0.1524" layer="91"/>
+<wire x1="302.26" y1="55.88" x2="302.26" y2="40.64" width="0.1524" layer="91"/>
+<junction x="302.26" y="40.64"/>
+<pinref part="U$12" gate="1" pin="1"/>
 </segment>
 </net>
@@
 <wire x1="254" y1="-10.16" x2="254" y2="-43.18" width="0.1524" layer="91"/>
 <pinref part="LED3" gate="G$1" pin="A"/>
+<pinref part="JP3" gate="A" pin="5"/>
+<wire x1="254" y1="-43.18" x2="162.56" y2="-43.18" width="0.1524" layer="91"/>
+<wire x1="162.56" y1="-43.18" x2="162.56" y2="2.54" width="0.1524" layer="91"/>
+<junction x="254" y="-43.18"/>
 </segment>
 </net>
@@
 <wire x1="259.08" y1="-7.62" x2="248.92" y2="-7.62" width="0.1524" layer="91"/>
 <wire x1="259.08" y1="-33.02" x2="259.08" y2="-7.62" width="0.1524" layer="91"/>
-<wire x1="259.08" y1="-33.02" x2="162.56" y2="-33.02" width="0.1524" layer="91"/>
+<wire x1="259.08" y1="-33.02" x2="231.14" y2="-33.02" width="0.1524" layer="91"/>
 <pinref part="JP2" gate="G$1" pin="2"/>
-</segment>
-</net>
+<wire x1="193.04" y1="2.54" x2="193.04" y2="-33.02" width="0.1524" layer="91"/>
+<wire x1="193.04" y1="-33.02" x2="231.14" y2="-33.02" width="0.1524" layer="91"/>
+<junction x="231.14" y="-33.02"/>
+<pinref part="JP3" gate="A" pin="6"/>
+<wire x1="193.04" y1="2.54" x2="170.18" y2="2.54" width="0.1524" layer="91"/>
+</segment>
+</net>
+<net name="N$3" class="0">
+<segment>
+<pinref part="JP3" gate="A" pin="3"/>
+<wire x1="162.56" y1="5.08" x2="157.48" y2="5.08" width="0.1524" layer="91"/>
+<wire x1="157.48" y1="5.08" x2="157.48" y2="-86.36" width="0.1524" layer="91"/>
+<pinref part="JP8" gate="A" pin="4_PWM"/>
+<wire x1="157.48" y1="-86.36" x2="264.16" y2="-86.36" width="0.1524" layer="91"/>
+</segment>
+</net>
+<net name="N$4" class="0">
+<segment>
+<pinref part="J4" gate="J1" pin="D+"/>
+<wire x1="294.64" y1="129.54" x2="254" y2="129.54" width="0.1524" layer="91"/>
+<pinref part="JP4" gate="A" pin="2"/>
+</segment>
+</net>
+<net name="N$6" class="0">
+<segment>
+<pinref part="J4" gate="J1" pin="D-"/>
+<wire x1="294.64" y1="127" x2="254" y2="127" width="0.1524" layer="91"/>
+<pinref part="JP4" gate="A" pin="4"/>
+</segment>
+</net>
+<net name="N$7" class="0">
+<segment>
+<pinref part="JP4" gate="A" pin="1"/>
+<wire x1="246.38" y1="129.54" x2="236.22" y2="129.54" width="0.1524" layer="91"/>
+<wire x1="236.22" y1="129.54" x2="236.22" y2="127" width="0.1524" layer="91"/>
+<pinref part="JP4" gate="A" pin="3"/>
+<wire x1="236.22" y1="127" x2="246.38" y2="127" width="0.1524" layer="91"/>
+<pinref part="JP3" gate="A" pin="4"/>
+<wire x1="177.8" y1="5.08" x2="170.18" y2="5.08" width="0.1524" layer="91"/>
+<pinref part="U$12" gate="1" pin="2"/>
+<wire x1="177.8" y1="5.08" x2="177.8" y2="58.42" width="0.1524" layer="91"/>
+<wire x1="177.8" y1="58.42" x2="254" y2="58.42" width="0.1524" layer="91"/>
+<wire x1="236.22" y1="129.54" x2="177.8" y2="129.54" width="0.1524" layer="91"/>
+<wire x1="177.8" y1="129.54" x2="177.8" y2="58.42" width="0.1524" layer="91"/>
+<junction x="236.22" y="129.54"/>
+<junction x="177.8" y="58.42"/>
+</segment>
+</net>
