File: pcb/daughterboard.brd (EAGLE design)
At the start: 28 x 24 mm, 27 parts, among them IC3 STM32F042F4, SW1 324_SW, SW2 324_SW, SW4 324_SW, SW5 324_SW, SW6 324_SW, U4 XC6206_DEV

Commit message: finishing touches before production run
Parts:
- removed SW6: 324_SW, 3pos_slide_switch_centered:342_SWICH_FOOT
- added SW3: 324_SW, 3pos_slide_switch_centered:342_SWICH_FOOT
- C1, C2: value 1uF -> 2.2uF
- moved U$4 17.2 mm to (17.4, 22.9), turned to 0 degrees
- moved U$1 12.8 mm to (26.8, 14.2), turned to 90 degrees
- moved U$7 10.1 mm to (26.8, 8.51), turned to 270 degrees
- moved SW5 10.0 mm to (17.4, 6.35), turned to 180 degrees
- moved SW1 8.36 mm to (23.6, 14.2), turned to 90 degrees
- moved U$8 7.72 mm to (18.3, 3.05), turned to 0 degrees
- moved U$3 6.48 mm to (23.7, 8.51)
- moved R1 5.97 mm to (2.41, 10.2), turned to 180 degrees
- moved R2 5.97 mm to (8.38, 10.2), turned to 0 degrees
- renumbered C4 to C3, IC3 to IC1, J4 to J1, JP3 to JP2, LED2 to LED1, R6 to R4, U4 to U1
Connections:
- net +3V3: now also U$7.1; no longer U$4.1
- net BUTTON1: now also U$3.1; no longer U$8.1
- net BUTTON2: now also U$7.2; no longer U$4.2
- net GND: now also SW3.P$1, SW3.P$4, SW5.P$2, SW5.P$3, U$4.2, U$8.1; no longer SW5.P$1, SW5.P$4, SW6.P$2, SW6.P$3, U$7.1, U$8.2
- net N$11: now also SW1.P$2, SW1.P$3, U$1.1; no longer SW5.P$2, SW5.P$3, U$3.1
- net N$12: now also SW5.P$1, SW5.P$4, U$8.2; no longer SW6.P$1, SW6.P$4, U$7.2
- net N$31: now also R2.1; no longer R1.1
- net N$33: now also R1.1; no longer R2.1
- net N$9: now also SW3.P$2, SW3.P$3, U$4.1; no longer SW1.P$2, SW1.P$3, U$1.1
