File: pcb/atx4vc.brd (EAGLE design)
At the start: 69 x 69 mm, 52 parts, among them IC1 MY_7905DT, J2 ATX24RH

Commit message: new production run
Parts:
- added TP2: TPTP12R, testpad:TP12R
Connections:
- net N$2: now also TP2.TP
Changed lines of the file:
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@@
 <layer number="14" name="Route14" color="22" fill="1" visible="no" active="no"/>
 <layer number="15" name="Route15" color="23" fill="1" visible="no" active="no"/>
-<layer number="16" name="Bottom" color="1" fill="1" visible="no" active="yes"/>
+<layer number="16" name="Bottom" color="1" fill="1" visible="yes" active="yes"/>
 <layer number="17" name="Pads" color="2" fill="1" visible="yes" active="yes"/>
 <layer number="18" name="Vias" color="2" fill="1" visible="yes" active="yes"/>
 <layer number="19" name="Unrouted" color="6" fill="1" visible="yes" active="yes"/>
 <layer number="20" name="Dimension" color="24" fill="1" visible="yes" active="yes"/>
-<layer number="21" name="tPlace" color="7" fill="1" visible="no" active="yes"/>
-<layer number="22" name="bPlace" color="7" fill="1" visible="no" active="yes"/>
+<layer number="21" name="tPlace" color="7" fill="1" visible="yes" active="yes"/>
+<layer number="22" name="bPlace" color="7" fill="1" visible="yes" active="yes"/>
 <layer number="23" name="tOrigins" color="15" fill="1" visible="yes" active="yes"/>
-<layer number="24" name="bOrigins" color="15" fill="1" visible="no" active="yes"/>
-<layer number="25" name="tNames" color="7" fill="1" visible="no" active="yes"/>
-<layer number="26" name="bNames" color="7" fill="1" visible="no" active="yes"/>
-<layer number="27" name="tValues" color="7" fill="1" visible="no" active="yes"/>
-<layer number="28" name="bValues" color="7" fill="1" visible="no" active="yes"/>
+<layer number="24" name="bOrigins" color="15" fill="1" visible="yes" active="yes"/>
+<layer number="25" name="tNames" color="7" fill="1" visible="yes" active="yes"/>
+<layer number="26" name="bNames" color="7" fill="1" visible="yes" active="yes"/>
+<layer number="27" name="tValues" color="7" fill="1" visible="yes" active="yes"/>
+<layer number="28" name="bValues" color="7" fill="1" visible="yes" active="yes"/>
 <layer number="29" name="tStop" color="7" fill="3" visible="no" active="yes"/>
 <layer number="30" name="bStop" color="7" fill="6" visible="no" active="yes"/>
@@
 <layer number="38" name="bTest" color="7" fill="1" visible="no" active="yes"/>
 <layer number="39" name="tKeepout" color="4" fill="11" visible="yes" active="yes"/>
-<layer number="40" name="bKeepout" color="1" fill="11" visible="no" active="yes"/>
+<layer number="40" name="bKeepout" color="1" fill="11" visible="yes" active="yes"/>
 <layer number="41" name="tRestrict" color="4" fill="10" visible="yes" active="yes"/>
-<layer number="42" name="bRestrict" color="1" fill="10" visible="no" active="yes"/>
+<layer number="42" name="bRestrict" color="1" fill="10" visible="yes" active="yes"/>
 <layer number="43" name="vRestrict" color="2" fill="10" visible="no" active="yes"/>
 <layer number="44" name="Drills" color="7" fill="1" visible="no" active="yes"/>
-<layer number="45" name="Holes" color="7" fill="1" visible="yes" active="yes"/>
+<layer number="45" name="Holes" color="7" fill="1" visible="no" active="yes"/>
 <layer number="46" name="Milling" color="3" fill="1" visible="yes" active="yes"/>
 <layer number="47" name="Measures" color="7" fill="1" visible="no" active="yes"/>
@@
 <layer number="49" name="Reference" color="7" fill="1" visible="no" active="yes"/>
 <layer number="50" name="dxf" color="7" fill="1" visible="no" active="no"/>
-<layer number="51" name="tDocu" color="7" fill="1" visible="no" active="yes"/>
-<layer number="52" name="bDocu" color="7" fill="1" visible="no" active="yes"/>
+<layer number="51" name="tDocu" color="7" fill="1" visible="yes" active="yes"/>
+<layer number="52" name="bDocu" color="7" fill="1" visible="yes" active="yes"/>
 <layer number="53" name="tGND_GNDA" color="7" fill="1" visible="no" active="no"/>
 <layer number="54" name="bGND_GNDA" color="7" fill="1" visible="no" active="no"/>
@@
 <attribute name="TP_SIGNAL_NAME" value="" x="58.0175" y="10.4" size="1.778" layer="28" rot="MR0" display="off"/>
 </element>
+<element name="TP2" library="testpad" library_urn="urn:adsk.eagle:library:385" package="TP12R" package3d_urn="urn:adsk.eagle:package:27963/1" value="TPTP12R" x="57.658" y="12.192" smashed="yes" rot="MR0">
+<attribute name="POPULARITY" value="1" x="57.658" y="12.192" size="1.778" layer="28" rot="MR0" display="off"/>
+<attribute name="TP_SIGNAL_NAME" value="" x="57.658" y="12.192" size="1.778" layer="28" rot="MR0" display="off"/>
+</element>
 </elements>
 <signals>
@@
 <wire x1="61.3605" y1="13.851" x2="61.3485" y2="13.839" width="0.2032" layer="1"/>
 <contactref element="JP1" pad="1"/>
-<wire x1="56.0239" y1="12.1" x2="58.2175" y2="12.1" width="0.2032" layer="16"/>
-<wire x1="58.2175" y1="12.1" x2="59.0175" y2="12.9" width="0.2032" layer="16"/>
 <via x="59.0175" y="12.9" extent="1-16" drill="0.5"/>
 <wire x1="59.9565" y1="13.839" x2="61.3485" y2="13.839" width="0.1524" layer="1"/>
 <wire x1="59.0175" y1="12.9" x2="59.9565" y2="13.839" width="0.1524" layer="1"/>
+<contactref element="TP2" pad="TP"/>
+<wire x1="56.0239" y1="12.1" x2="57.566" y2="12.1" width="0.254" layer="16"/>
+<wire x1="57.566" y1="12.1" x2="57.658" y2="12.192" width="0.254" layer="16"/>
+<wire x1="57.658" y1="12.192" x2="58.366" y2="12.9" width="0.254" layer="16"/>
+<wire x1="58.366" y1="12.9" x2="59.0175" y2="12.9" width="0.254" layer="16"/>
 </signal>
 <signal name="N$4">
