File: pcb/atx4vc.sch (EAGLE design)
At the start: 49 parts, among them IC1 MY_7905DT, J2 ATX24RH

Commit message: minor adjustments for next production run
Parts:
- added JP1, JP6: JUMPER-SMT_2_NO_NO-SILK, SparkFun-Jumpers:JUMPER-SMT_2_NO_NO-SILK
- added TP1: TPTP12R, testpad:TPTP12R
Connections:
- new net N$2: J1.D+, JP1.1
- new net N$4: J1.D-, JP6.1, TP1.TP
- net N$7: now also JP1.2, JP6.2; no longer J1.D+
Changed lines of the file:
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@@
 <part name="GND23" library="supply1" deviceset="GND" device=""/>
 <part name="U$13" library="adafruit_changed" deviceset="PINHD1X2" device=""/>
+<part name="JP1" library="SparkFun-Jumpers" deviceset="JUMPER-SMT_2_NO" device="_NO-SILK"/>
+<part name="JP6" library="SparkFun-Jumpers" deviceset="JUMPER-SMT_2_NO" device="_NO-SILK"/>
+<part name="TP1" library="testpad" library_urn="urn:adsk.eagle:library:385" deviceset="TP" device="TP12R" package3d_urn="urn:adsk.eagle:package:27963/1"/>
 </parts>
 <sheets>
@@
 <attribute name="NAME" x="318.77" y="79.375" size="1.778" layer="95"/>
 <attribute name="VALUE" x="318.77" y="68.58" size="1.778" layer="96"/>
+</instance>
+<instance part="JP1" gate="G$1" x="205.74" y="129.54" smashed="yes" rot="R180">
+<attribute name="NAME" x="208.28" y="127" size="1.778" layer="95" font="vector" rot="R180"/>
+<attribute name="VALUE" x="208.28" y="132.08" size="1.778" layer="96" font="vector" rot="R180" align="top-left"/>
+</instance>
+<instance part="JP6" gate="G$1" x="205.74" y="119.38" smashed="yes" rot="R180">
+<attribute name="NAME" x="208.28" y="116.84" size="1.778" layer="95" font="vector" rot="R180"/>
+<attribute name="VALUE" x="208.28" y="121.92" size="1.778" layer="96" font="vector" rot="R180" align="top-left"/>
+</instance>
+<instance part="TP1" gate="G$1" x="241.3" y="124.46" smashed="yes" rot="R180">
+<attribute name="NAME" x="242.57" y="123.19" size="1.778" layer="95" rot="R180"/>
+<attribute name="TP_SIGNAL_NAME" x="240.03" y="125.73" size="1.778" layer="97" rot="R180"/>
 </instance>
 </instances>
@@
 <wire x1="177.8" y1="5.08" x2="177.8" y2="58.42" width="0.1524" layer="91"/>
 <wire x1="177.8" y1="58.42" x2="254" y2="58.42" width="0.1524" layer="91"/>
-<wire x1="294.64" y1="129.54" x2="177.8" y2="129.54" width="0.1524" layer="91"/>
 <wire x1="177.8" y1="129.54" x2="177.8" y2="58.42" width="0.1524" layer="91"/>
 <junction x="177.8" y="58.42"/>
+<wire x1="200.66" y1="129.54" x2="195.58" y2="129.54" width="0.1524" layer="91"/>
+<pinref part="JP1" gate="G$1" pin="2"/>
+<pinref part="JP6" gate="G$1" pin="2"/>
+<wire x1="195.58" y1="129.54" x2="177.8" y2="129.54" width="0.1524" layer="91"/>
+<wire x1="200.66" y1="119.38" x2="195.58" y2="119.38" width="0.1524" layer="91"/>
+<wire x1="195.58" y1="119.38" x2="195.58" y2="129.54" width="0.1524" layer="91"/>
+<junction x="195.58" y="129.54"/>
+</segment>
+</net>
+<net name="N$2" class="0">
+<segment>
 <pinref part="J1" gate="J1" pin="D+"/>
-</segment>
-</net>
+<wire x1="294.64" y1="129.54" x2="210.82" y2="129.54" width="0.1524" layer="91"/>
+<pinref part="JP1" gate="G$1" pin="1"/>
+</segment>
+</net>
+<net name="N$4" class="0">
+<segment>
+<pinref part="J1" gate="J1" pin="D-"/>
+<pinref part="JP6" gate="G$1" pin="1"/>
+<wire x1="294.64" y1="127" x2="241.3" y2="127" width="0.1524" layer="91"/>
+<wire x1="241.3" y1="127" x2="210.82" y2="127" width="0.1524" layer="91"/>
+<wire x1="210.82" y1="127" x2="210.82" y2="119.38" width="0.1524" layer="91"/>
+<pinref part="TP1" gate="G$1" pin="TP"/>
+<junction x="241.3" y="127"/>
+</segment>
+</net>

Commit message: adjusted hole size
Parts:
- U$7: value VH396_8P -> 396_CONN_VH396_8P; device 396_conn:VH396_8P -> atx4vc:396_CONN_VH396_8P
Changed lines of the file:
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@@
 <part name="U$10" library="atx_power_control" deviceset="CAR_FUSE_HOLDER" device="3IN1"/>
 <part name="U$9" library="atx_power_control" deviceset="CAR_FUSE_HOLDER" device="3IN1"/>
-<part name="U$7" library="396_conn" deviceset="VH396_8P" device=""/>
+<part name="U$7" library="atx4vc" deviceset="396_CONN_VH396_8P" device=""/>
 <part name="GND37" library="backplane" deviceset="GND" device=""/>
 <part name="R2" library="atx_power_control" deviceset="RESISTOR" device="0805-RES" value="5K1"/>

Commit message: new production run
Parts:
- added TP2: TPTP12R, testpad:TPTP12R
Connections:
- net N$2: now also TP2.TP
Changed lines of the file:
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@@
 <part name="JP6" library="SparkFun-Jumpers" deviceset="JUMPER-SMT_2_NO" device="_NO-SILK"/>
 <part name="TP1" library="testpad" library_urn="urn:adsk.eagle:library:385" deviceset="TP" device="TP12R" package3d_urn="urn:adsk.eagle:package:27963/1"/>
+<part name="TP2" library="testpad" library_urn="urn:adsk.eagle:library:385" deviceset="TP" device="TP12R" package3d_urn="urn:adsk.eagle:package:27963/1"/>
 </parts>
 <sheets>
@@
 <attribute name="NAME" x="242.57" y="123.19" size="1.778" layer="95" rot="R180"/>
 <attribute name="TP_SIGNAL_NAME" x="240.03" y="125.73" size="1.778" layer="97" rot="R180"/>
+</instance>
+<instance part="TP2" gate="G$1" x="241.3" y="132.08" smashed="yes">
+<attribute name="NAME" x="240.03" y="133.35" size="1.778" layer="95"/>
+<attribute name="TP_SIGNAL_NAME" x="242.57" y="130.81" size="1.778" layer="97"/>
 </instance>
 </instances>
@@
 <segment>
 <pinref part="J1" gate="J1" pin="D+"/>
-<wire x1="294.64" y1="129.54" x2="210.82" y2="129.54" width="0.1524" layer="91"/>
+<wire x1="294.64" y1="129.54" x2="241.3" y2="129.54" width="0.1524" layer="91"/>
 <pinref part="JP1" gate="G$1" pin="1"/>
-</segment>
-</net>
+<pinref part="TP2" gate="G$1" pin="TP"/>
+<wire x1="241.3" y1="129.54" x2="210.82" y2="129.54" width="0.1524" layer="91"/>
+<junction x="241.3" y="129.54"/>
+</segment>
+</net>
