File: pcb/pt0/atx_power_control.brd (EAGLE design)
At the start: 100 x 70 mm, 59 parts, among them IC2 REG1117, IC3 STM32F042F4, IC4 MY_7905DT, J1 ATX24RH, SW1 324_SW, SW3 324_SW, SW4 324_SW, U2 USBC_16P

Commit message: adjusted pcb
Parts:
- moved R3 2.67 mm to (36.3, 13.7)
- moved LED3 2.67 mm to (32.0, 13.7)
Routing:
- net N$28: track 54.1 -> 56.7 mm
Other:
- board text added: "ATX CONTROL BOARD dekuNukem July 2022 PT0"
- board text added: "PWR OK"
- board text added: "PWR ON"
- board text removed: "ATX CONTROL BOARD dekuNukem AUG 2022 PT1"
- board text removed: "CLK"
- board text removed: "DIO"
- board text removed: "POK"
- board text removed: "PON"
- board text removed: "RX"
- board text removed: "TX"
Changed lines of the file:
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@@
 <text x="20.447" y="8.4282" size="1.6764" layer="25" rot="R180" align="center">5VSB</text>
 <text x="25.6832" y="8.382" size="1.6764" layer="25" align="center">G</text>
-<text x="35.4622" y="8.636" size="1.6764" layer="25" align="center">G</text>
-<text x="30.226" y="8.6822" size="1.6764" layer="25" rot="R180" align="center">POK</text>
+<text x="35.3352" y="8.636" size="1.6764" layer="25" align="center">G</text>
+<text x="31.115" y="9.9522" size="1.6764" layer="25" rot="R180" align="center">PWR
+OK</text>
 <text x="44.577" y="29.21" size="1.4224" layer="25" align="center">PWR
 SW</text>
-<text x="39.878" y="8.636" size="1.6764" layer="25" align="center">PON</text>
-<text x="44.4792" y="8.636" size="1.6764" layer="25" align="center">G</text>
+<text x="39.878" y="9.906" size="1.6764" layer="25" align="center">PWR
+ON</text>
+<text x="43.9712" y="8.636" size="1.6764" layer="25" align="center">G</text>
 <text x="4.953" y="6.9042" size="1.6764" layer="25" rot="R180" align="center">5VSB</text>
 <text x="69.7522" y="23.8714" size="1.4224" layer="25" align="center">G</text>
@@
 <text x="75.7212" y="26.7924" size="1.4224" layer="25" align="center">3V3</text>
 <text x="63.5" y="16.637" size="2.54" layer="25" rot="R180" align="center">ATX CONTROL BOARD
-dekuNukem AUG 2022
-PT1</text>
+dekuNukem July 2022
+PT0</text>
 <text x="45.466" y="38.354" size="1.27" layer="25" rot="R270" align="center">G</text>
 <text x="53.213" y="37.592" size="1.27" layer="25" rot="R270" align="center">PA0</text>
@@
 <rectangle x1="65.278" y1="0" x2="83.82" y2="12.573" layer="41"/>
 <rectangle x1="65.278" y1="0" x2="83.82" y2="12.573" layer="42"/>
-<text x="44.8602" y="53.8434" size="1.1684" layer="25" align="center">GND</text>
-<text x="39.3992" y="56.1294" size="1.143" layer="25" align="center">3V3</text>
-<text x="36.7322" y="51.1764" size="1.143" layer="25" align="center">TX</text>
-<text x="34.1922" y="56.2564" size="1.143" layer="25" align="center">DIO</text>
-<text x="31.6522" y="51.1764" size="1.143" layer="25" align="center">CLK</text>
-<text x="25.9372" y="53.8434" size="1.143" layer="25" align="center">RX</text>
 </plain>
 <attributes>
@@
 <attribute name="NAME" x="27.9527" y="67.7456" size="0.8128" layer="25" rot="R270"/>
 </element>
-<element name="LED3" library="adafruit" package="CHIP-LED0805" value="" x="29.591" y="12.573" smashed="yes" rot="R270">
-<attribute name="VALUE" x="28.321" y="10.033" size="1.27" layer="27"/>
-</element>
-<element name="R3" library="SparkFun-Passives" package="0805" value="1K" x="33.909" y="12.573" smashed="yes" rot="R180">
-<attribute name="NAME" x="36.8808" y="12.8905" size="0.8128" layer="25" rot="R180"/>
+<element name="LED3" library="adafruit" package="CHIP-LED0805" value="" x="32.004" y="13.716" smashed="yes" rot="R270">
+<attribute name="VALUE" x="30.734" y="11.176" size="1.27" layer="27"/>
+</element>
+<element name="R3" library="SparkFun-Passives" package="0805" value="1K" x="36.322" y="13.716" smashed="yes" rot="R180">
+<attribute name="NAME" x="39.2938" y="14.0335" size="0.8128" layer="25" rot="R180"/>
 </element>
 <element name="JP3" library="pinhead" library_urn="urn:adsk.eagle:library:325" package="1X06" package3d_urn="urn:adsk.eagle:package:22472/2" value="" x="35.415" y="53.78" smashed="yes">
@@
 </element>
 <element name="J8" library="SparkFun-Connectors" package="SCREWTERMINAL-3.5MM-2" value="" x="21.59" y="3.683" smashed="yes">
+<attribute name="NAME" x="20.32" y="6.223" size="0.6096" layer="25" font="vector" ratio="20"/>
 <attribute name="PROD_ID" value="CONN-08399" x="21.59" y="3.683" size="0.8128" layer="27" display="off"/>
 <attribute name="VALUE" x="20.32" y="4.953" size="0.6096" layer="27" font="vector" ratio="20"/>
 </element>
 <element name="J9" library="SparkFun-Connectors" package="SCREWTERMINAL-3.5MM-2" value="" x="30.988" y="3.683" smashed="yes">
+<attribute name="NAME" x="29.718" y="6.223" size="0.6096" layer="25" font="vector" ratio="20"/>
 <attribute name="PROD_ID" value="CONN-08399" x="30.988" y="3.683" size="0.8128" layer="27" display="off"/>
 <attribute name="VALUE" x="29.718" y="4.953" size="0.6096" layer="27" font="vector" ratio="20"/>
 </element>
 <element name="J10" library="SparkFun-Connectors" package="SCREWTERMINAL-3.5MM-2" value="" x="40.386" y="3.683" smashed="yes">
+<attribute name="NAME" x="39.116" y="6.223" size="0.6096" layer="25" font="vector" ratio="20"/>
 <attribute name="PROD_ID" value="CONN-08399" x="40.386" y="3.683" size="0.8128" layer="27" display="off"/>
 <attribute name="VALUE" x="39.116" y="4.953" size="0.6096" layer="27" font="vector" ratio="20"/>
@@
 <contactref element="LED3" pad="C"/>
 <contactref element="R3" pad="2"/>
-<wire x1="30.641" y1="12.573" x2="33.009" y2="12.573" width="0.4064" layer="1"/>
+<wire x1="33.054" y1="13.716" x2="35.422" y2="13.716" width="0.4064" layer="1"/>
 </signal>
 <signal name="N$3">
@@
 <wire x1="16.5608" y1="11.2268" x2="18.8976" y2="8.89" width="0.4064" layer="1"/>
 <contactref element="LED3" pad="A"/>
-<wire x1="28.541" y1="12.573" x2="28.575" y2="12.539" width="0.4064" layer="1"/>
-<wire x1="28.575" y1="12.539" x2="28.575" y2="8.89" width="0.4064" layer="1"/>
-<wire x1="18.8976" y1="8.89" x2="28.575" y2="8.89" width="0.4064" layer="1"/>
-<wire x1="30.988" y1="3.683" x2="30.988" y2="6.477" width="0.4064" layer="1"/>
-<wire x1="30.988" y1="6.477" x2="28.575" y2="8.89" width="0.4064" layer="1"/>
+<wire x1="30.954" y1="13.716" x2="30.988" y2="13.682" width="0.4064" layer="1"/>
+<wire x1="30.988" y1="13.682" x2="30.988" y2="8.89" width="0.4064" layer="1"/>
+<wire x1="30.988" y1="8.89" x2="30.988" y2="3.683" width="0.4064" layer="1"/>
+<wire x1="18.8976" y1="8.89" x2="30.988" y2="8.89" width="0.4064" layer="1"/>
 </signal>
 <signal name="N$27">
