File: pcb/pt1/atx_power_control.brd (EAGLE design)
At the start: 86 x 70 mm, 55 parts, among them IC2 REG1117, IC3 STM32F042F4, IC4 MY_7905DT, J1 ATX24RH, SW1 324_SW, SW3 324_SW, SW4 324_SW, U2 USBC_16P

Commit message: working on new ATX PCB
Parts:
- added IC1: (no value), linear:TO220H
- added JP8: (no value), pinhead:1X04
- added JP9: (no value), pinhead:1X03
- added R13: (no value), SparkFun-Retired:TRIM_POT_PTH
- JP1: device pinhead:1X02/90 -> pinhead:1X04
- moved R6 137.0 mm to (5.31, 2.24)
- moved LED2 123.7 mm to (5.29, 4.48)
- moved J8 105.8 mm to (21.6, 3.68)
- moved R3 102.7 mm to (33.9, 12.6)
- moved LED3 102.0 mm to (29.6, 12.6)
- moved J9 98.8 mm to (31.0, 3.68)
- moved J10 79.4 mm to (40.4, 3.68)
- moved JP1 52.8 mm to (73.7, 66.0)
- moved JP4 28.0 mm to (69.6, 58.2)
- moved R5 26.2 mm to (25.4, 36.9)
- moved C27 25.1 mm to (51.1, 10.5), turned to 0 degrees
- moved SW3 20.9 mm to (30.1, 41.4)
- moved JP7 19.1 mm to (49.3, 48.8)
- moved JP5 19.0 mm to (29.3, 29.3)
- moved C5 18.3 mm to (57.5, 9.53), turned to 0 degrees
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Connections:
- new net N$14: IC3.11, JP1.3, JP7.4
- new net N$17: JP1.2, JP2.2, JP4.2
- new net N$21: IC3.12, JP1.4, JP7.3
- new net N$22: IC3.13, JP2.3, JP7.2
- new net N$23: IC3.14, JP2.4, JP7.1
- new net N$27: IC3.6, JP8.4, R13.2
- new net N$30: IC3.7, JP8.3
- new net N$32: IC3.10, JP8.2
- net +3V3: now also R13.1
- net GND: now also IC1.1, JP1.1, JP2.1, JP8.1, R13.3
- net N$11: now also IC1.3
- net N$15: now also JP9.1
- net N$19: now also JP9.3; no longer JP1.2
- net N$2: now also IC1.2
- net N$34: now also JP9.2; no longer JP1.1
Routing:
- net N$2: track 0.00 -> 114.1 mm
- net N$12: track 0.00 -> 112.8 mm
- net VCC: track 0.00 -> 109.7 mm
- net N$10: track 0.00 -> 81.6 mm
- net N$13: track 0.00 -> 64.0 mm
- net N$15: track 0.00 -> 61.0 mm
- net N$28: track 0.00 -> 54.1 mm
- net N$11: track 0.00 -> 47.2 mm
- net N$14: track 0.00 -> 44.4 mm
- net N$26: track 0.00 -> 43.7 mm
- net N$21: track 0.00 -> 43.2 mm
- net N$6: track 0.00 -> 35.8 mm
- net N$22: track 0.00 -> 31.9 mm
- net GND: track 0.00 -> 31.8 mm
- net N$16: track 0.00 -> 31.7 mm
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Other:
- board size 86 x 70 mm -> 100 x 70 mm
