File: pcb/pt1/atx_power_control.sch (EAGLE design)
At the start: 55 parts, among them IC2 REG1117, IC3 STM32F042F4, IC4 MY_7905DT, J1 ATX24RH, SW1 324_SW, SW3 324_SW, SW4 324_SW, U2 USBC_16P

Commit message: working on new ATX PCB
Parts:
- added IC1: (no value), linear:7905T
- added JP8: (no value), pinhead:PINHD-1X4
- added JP9: (no value), pinhead:PINHD-1X3
- added R13: (no value), SparkFun-Retired:TRIMPOTPTH
- JP1: device pinhead:PINHD-1X2/90 -> pinhead:PINHD-1X4
Connections:
- new net N$14: IC3.PA5, JP1.3, JP7.4
- new net N$17: JP1.2, JP2.2, JP4.2
- new net N$21: IC3.PA6, JP1.4, JP7.3
- new net N$22: IC3.PA7, JP2.3, JP7.2
- new net N$23: IC3.PB1, JP2.4, JP7.1
- new net N$27: IC3.PA0, JP8.4, R13.WIPER
- new net N$30: IC3.PA1, JP8.3
- new net N$32: IC3.PA4, JP8.2
- net +3V3: now also R13.CCW
- net GND: now also IC1.GND, JP1.1, JP2.1, JP8.1, R13.CW
- net N$11: now also IC1.VO
- net N$15: now also JP9.1
- net N$19: now also JP9.3; no longer JP1.2
- net N$2: now also IC1.VI
- net N$34: now also JP9.2; no longer JP1.1
Other:
- moved on the sheet: JP2, JP7
