File: pcb/pt2/atx_power_control.brd (EAGLE design)
At the start: 86 x 70 mm, 57 parts, among them IC2 REG1117, IC3 STM32F042F4, IC4 MY_7905DT, J1 ATX24RH, SW1 324_SW, SW2 324_SW, SW3 324_SW, SW4 324_SW, U2 USBC_16P

Commit message: updated atx board
Parts:
- removed J5, J8: (no value), atx_power_control:SCREWTERMINAL-3.5MM-2
- J7: device atx_power_control:SCREWTERMINAL-3.5MM-2-NS -> atx_power_control:SCREWTERMINAL-3.5MM-2
- moved SW1 6.37 mm to (24.9, 13.2)
Connections:
- net GND: no longer J5.2
- net N$17: no longer J8.1
- net N$19: no longer J8.2
- net N$26: no longer J5.1
Routing:
- net N$19: track 45.5 -> 37.1 mm
- net N$17: track 11.8 -> 3.81 mm
- net N$26: track 28.5 -> 25.8 mm
- net GND: track 18.2 -> 15.6 mm
Other:
- board text added: "ATX CONTROL BOARD dekuNukem AUG 2022 PT2"
- board text removed: "ATX CONTROL BOARD dekuNukem AUG 2022 PT3"
Changed lines of the file:
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@@
 <text x="22.86" y="35.179" size="1.4224" layer="25" rot="R270" align="center">DFU</text>
 <text x="33.655" y="35.306" size="1.4224" layer="25" rot="R270" align="center">RST</text>
-<text x="24.13" y="11.176" size="1.778" layer="25" align="center">PWR
+<text x="30.988" y="11.049" size="1.778" layer="25" align="center">PWR
 SW</text>
 <circle x="4.318" y="4.191" radius="4" width="0" layer="41"/>
@@
 <text x="6.096" y="35.052" size="2.54" layer="26" rot="MR90" align="center">ATX CONTROL BOARD
 dekuNukem AUG 2022
-PT3</text>
+PT2</text>
 <text x="43.9712" y="42.7944" size="1.1684" layer="25" align="center">GND</text>
 <text x="41.3042" y="48.0014" size="1.143" layer="25" align="center">3V3</text>
@@
 <text x="62.2254" y="58.1368" size="1.4224" layer="25" rot="R270" align="center">5V</text>
 <text x="64.7654" y="58.2638" size="1.4224" layer="25" rot="R270" align="center">DATA</text>
-<text x="65.405" y="22.733" size="1.4224" layer="25" rot="R180" align="center">PWR
+<text x="61.214" y="11.176" size="1.778" layer="25" rot="R180" align="center">PWR
 LED</text>
-<text x="65.024" y="10.414" size="3.81" layer="25" rot="R180" align="center">+</text>
+<text x="64.516" y="22.733" size="3.81" layer="25" rot="R180" align="center">+</text>
 <text x="31.2712" y="48.0014" size="1.143" layer="25" align="center">PG</text>
 <text x="34.798" y="14.097" size="1.4224" layer="25" rot="R270" align="center">COLOR/SPD</text>
 <text x="34.798" y="25.908" size="1.4224" layer="25" rot="R270" align="center">BRIGHT</text>
 <text x="57.404" y="17.907" size="1.4224" layer="25" rot="R270" align="center">FAN SPD</text>
-<text x="56.388" y="11.43" size="1.016" layer="25" rot="R180" align="center">RGB
+<text x="56.642" y="11.557" size="1.016" layer="25" align="center">RGB
 MODE</text>
 <text x="25.8618" y="47.879" size="1.4224" layer="25" rot="R270" align="center">5VSB</text>
@@
 <attribute name="VALUE" x="84.074" y="58.928" size="0.6096" layer="27" font="vector" ratio="20" rot="R270"/>
 </element>
-<element name="J7" library="atx_power_control" package="SCREWTERMINAL-3.5MM-2-NS" value="" x="82.804" y="47.498" smashed="yes" rot="R270">
+<element name="J7" library="atx_power_control" package="SCREWTERMINAL-3.5MM-2" value="" x="82.804" y="47.498" smashed="yes" rot="R270">
 <attribute name="PROD_ID" value="CONN-08399" x="82.804" y="47.498" size="1.778" layer="27" rot="R270" display="off"/>
 <attribute name="VALUE" x="84.074" y="48.768" size="0.6096" layer="27" font="vector" ratio="20" rot="R270"/>
@@
 <element name="IC4" library="atx_power_control" package="ADAFRUIT_TO252" value="MY_7905DT" x="70.104" y="14.478" smashed="yes" rot="R180"/>
 <element name="C5" library="clock" package="0805@1" value="1uF" x="65.405" y="18.542" smashed="yes" rot="R90">
-<attribute name="NAME" x="65.7225" y="15.875" size="0.8128" layer="25" rot="R90"/>
+<attribute name="NAME" x="65.8495" y="15.494" size="0.8128" layer="25" rot="R90"/>
 </element>
 <element name="LED4" library="adafruit" package="CHIP-LED0805" value="" x="75.946" y="16.637" smashed="yes" rot="R90">
@@
 <attribute name="VALUE" x="31.115" y="31.623" size="1.27" layer="27" rot="R180"/>
 </element>
-<element name="SW1" library="3pos_slide_switch_centered" package="342_SWICH_FOOT" value="324_SW" x="25.4" y="19.558" smashed="yes" rot="R270"/>
+<element name="SW1" library="3pos_slide_switch_centered" package="342_SWICH_FOOT" value="324_SW" x="24.892" y="13.208" smashed="yes" rot="R270"/>
 <element name="JP6" library="pinhead" library_urn="urn:adsk.eagle:library:325" package="1X02" package3d_urn="urn:adsk.eagle:package:22435/2" value="" x="30.988" y="19.812" smashed="yes" rot="R180">
 <attribute name="POPULARITY" value="98" x="30.988" y="19.812" size="1.778" layer="27" rot="R180" display="off"/>
@@
 </element>
 <element name="R12" library="joyAnalog" package="0805" value="300" x="47.117" y="11.43" smashed="yes" rot="R90">
-<attribute name="NAME" x="45.5295" y="10.414" size="0.8128" layer="25" rot="R90"/>
-</element>
-<element name="J5" library="atx_power_control" package="SCREWTERMINAL-3.5MM-2" value="" x="28.575" y="12.192" smashed="yes">
-<attribute name="PROD_ID" value="CONN-08399" x="28.575" y="12.192" size="1.778" layer="27" display="off"/>
-<attribute name="VALUE" x="27.305" y="13.462" size="0.6096" layer="27" font="vector" ratio="20"/>
-</element>
-<element name="J8" library="atx_power_control" package="SCREWTERMINAL-3.5MM-2" value="" x="60.452" y="12.192" smashed="yes">
-<attribute name="PROD_ID" value="CONN-08399" x="60.452" y="12.192" size="1.778" layer="27" display="off"/>
-<attribute name="VALUE" x="59.182" y="13.462" size="0.6096" layer="27" font="vector" ratio="20"/>
+<attribute name="NAME" x="47.4345" y="13.208" size="0.8128" layer="25" rot="R90"/>
 </element>
 </elements>
@@
 <contactref element="U$5" pad="A"/>
 <contactref element="R12" pad="2"/>
-<contactref element="J5" pad="2"/>
-<wire x1="67.31" y1="50.038" x2="69.85" y2="50.038" width="2.2352" layer="1"/>
 </signal>
 <signal name="+3V3">
@@
 <wire x1="64.7065" y1="22.733" x2="62.484" y2="20.5105" width="0.3048" layer="1"/>
 <wire x1="62.484" y1="20.5105" x2="62.484" y2="19.939" width="0.3048" layer="1"/>
-<contactref element="J8" pad="2"/>
-<wire x1="62.484" y1="19.939" x2="63.119" y2="19.304" width="0.2032" layer="1"/>
-<wire x1="63.119" y1="19.304" x2="63.119" y2="13.025" width="0.2032" layer="1"/>
-<wire x1="63.119" y1="13.025" x2="63.952" y2="12.192" width="0.2032" layer="1"/>
 </signal>
 <signal name="N$24">
@@
 <contactref element="SW1" pad="P$3"/>
 <wire x1="37.46" y1="31.5132" x2="37.46" y2="28.56985625" width="0.2032" layer="1"/>
-<wire x1="26.525" y1="17.358" x2="26.525" y2="19.812" width="1.016" layer="1"/>
+<wire x1="26.017" y1="11.008" x2="26.017" y2="15.408" width="1.016" layer="1"/>
 <contactref element="JP6" pad="2"/>
-<wire x1="26.525" y1="19.812" x2="26.525" y2="21.758" width="1.016" layer="1"/>
-<wire x1="29.718" y1="20.82785625" x2="37.46" y2="28.56985625" width="0.2032" layer="1"/>
-<wire x1="29.718" y1="19.812" x2="29.718" y2="20.82785625" width="0.2032" layer="1"/>
-<contactref element="J5" pad="1"/>
-<wire x1="29.718" y1="19.812" x2="26.525" y2="19.812" width="0.2032" layer="1"/>
-<wire x1="26.525" y1="17.358" x2="26.525" y2="14.242" width="0.2032" layer="1"/>
-<wire x1="26.525" y1="14.242" x2="28.575" y2="12.192" width="0.2032" layer="1"/>
+<wire x1="37.46" y1="28.56985625" x2="32.00414375" y2="23.114" width="0.2032" layer="1"/>
+<wire x1="32.00414375" y1="23.114" x2="30.988" y2="23.114" width="0.2032" layer="1"/>
+<wire x1="29.718" y1="21.844" x2="30.988" y2="23.114" width="0.2032" layer="1"/>
+<wire x1="29.718" y1="19.812" x2="29.718" y2="21.844" width="0.2032" layer="1"/>
+<wire x1="29.718" y1="19.812" x2="29.718" y2="19.109" width="0.2032" layer="1"/>
+<wire x1="29.718" y1="19.109" x2="26.017" y2="15.408" width="0.2032" layer="1"/>
 </signal>
 <signal name="N$28">
@@
 <wire x1="59.955" y1="23.749" x2="59.955" y2="19.95" width="0.2032" layer="1"/>
 <wire x1="59.955" y1="19.95" x2="59.944" y2="19.939" width="0.2032" layer="1"/>
-<contactref element="J8" pad="1"/>
-<wire x1="59.944" y1="19.939" x2="59.944" y2="12.7" width="0.2032" layer="1"/>
-<wire x1="59.944" y1="12.7" x2="60.452" y2="12.192" width="0.2032" layer="1"/>
 </signal>
 <signal name="N$21">
