File: pcb/pt2/atx_power_control.sch (EAGLE design)
At the start: 57 parts, among them IC2 REG1117, IC3 STM32F042F4, IC4 MY_7905DT, J1 ATX24RH, SW1 324_SW, SW2 324_SW, SW3 324_SW, SW4 324_SW, U2 USBC_16P

Commit message: updated atx board
Parts:
- removed J5, J8: (no value), atx_power_control:CONN_023.5MM
- J7: device atx_power_control:CONN_023.5MM-NO_SILK -> atx_power_control:CONN_023.5MM
Connections:
- net GND: no longer J5.2
- net N$17: no longer J8.1
- net N$19: no longer J8.2
- net N$26: no longer J5.1
Changed lines of the file:
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@@
 <part name="J1" library="SparkFun-Connectors" deviceset="ATX24" device="RH"/>
 <part name="J6" library="atx_power_control" deviceset="CONN_02" device="3.5MM"/>
-<part name="J7" library="atx_power_control" deviceset="CONN_02" device="3.5MM-NO_SILK"/>
+<part name="J7" library="atx_power_control" deviceset="CONN_02" device="3.5MM"/>
 <part name="J2" library="atx_power_control" deviceset="CONN_02" device="3.5MM"/>
 <part name="J3" library="atx_power_control" deviceset="CONN_02" device="3.5MM"/>
@@
 <part name="R12" library="joyAnalog" deviceset="RESISTOR" device="0805-RES" value="300"/>
 <part name="GND35" library="backplane" deviceset="GND" device=""/>
-<part name="J5" library="atx_power_control" deviceset="CONN_02" device="3.5MM"/>
-<part name="J8" library="atx_power_control" deviceset="CONN_02" device="3.5MM"/>
 </parts>
 <sheets>
@@
 <instance part="GND35" gate="1" x="-139.7" y="-5.08" smashed="yes">
 <attribute name="VALUE" x="-142.24" y="-7.62" size="1.778" layer="96"/>
-</instance>
-<instance part="J5" gate="G$1" x="55.88" y="-7.62" smashed="yes" rot="R180">
-<attribute name="VALUE" x="58.42" y="-2.794" size="1.778" layer="96" font="vector" rot="R180"/>
-<attribute name="NAME" x="58.42" y="-13.208" size="1.778" layer="95" font="vector" rot="R180"/>
-</instance>
-<instance part="J8" gate="G$1" x="330.2" y="50.8" smashed="yes" rot="R180">
-<attribute name="VALUE" x="332.74" y="55.626" size="1.778" layer="96" font="vector" rot="R180"/>
-<attribute name="NAME" x="332.74" y="45.212" size="1.778" layer="95" font="vector" rot="R180"/>
 </instance>
 </instances>
@@
 <pinref part="JP6" gate="G$1" pin="1"/>
 <wire x1="17.78" y1="-10.16" x2="33.02" y2="-10.16" width="0.1524" layer="91"/>
-<pinref part="J5" gate="G$1" pin="2"/>
-<wire x1="48.26" y1="-10.16" x2="33.02" y2="-10.16" width="0.1524" layer="91"/>
-<junction x="33.02" y="-10.16"/>
 </segment>
 <segment>
@@
 <pinref part="J2" gate="G$1" pin="2"/>
 <wire x1="292.1" y1="22.86" x2="314.96" y2="22.86" width="0.1524" layer="91"/>
-<wire x1="314.96" y1="22.86" x2="347.98" y2="22.86" width="0.1524" layer="91"/>
+<wire x1="317.5" y1="22.86" x2="347.98" y2="22.86" width="0.1524" layer="91"/>
 <wire x1="347.98" y1="22.86" x2="368.3" y2="22.86" width="0.1524" layer="91"/>
 <wire x1="368.3" y1="22.86" x2="368.3" y2="25.4" width="0.1524" layer="91"/>
 <junction x="347.98" y="22.86"/>
 <pinref part="JP1" gate="G$1" pin="1"/>
-<wire x1="314.96" y1="55.88" x2="314.96" y2="48.26" width="0.1524" layer="91"/>
-<wire x1="314.96" y1="48.26" x2="314.96" y2="22.86" width="0.1524" layer="91"/>
-<pinref part="J8" gate="G$1" pin="2"/>
-<wire x1="322.58" y1="48.26" x2="314.96" y2="48.26" width="0.1524" layer="91"/>
-<junction x="314.96" y="48.26"/>
+<wire x1="314.96" y1="55.88" x2="314.96" y2="22.86" width="0.1524" layer="91"/>
+<wire x1="314.96" y1="22.86" x2="317.5" y2="22.86" width="0.1524" layer="91"/>
 </segment>
 </net>
@@
 <wire x1="33.02" y1="-7.62" x2="10.16" y2="-7.62" width="0.1524" layer="91"/>
 <junction x="10.16" y="-7.62"/>
-<pinref part="J5" gate="G$1" pin="1"/>
-<wire x1="33.02" y1="-7.62" x2="48.26" y2="-7.62" width="0.1524" layer="91"/>
-<junction x="33.02" y="-7.62"/>
 </segment>
 </net>
@@
 <pinref part="JP1" gate="G$1" pin="2"/>
 <wire x1="317.5" y1="63.5" x2="317.5" y2="55.88" width="0.1524" layer="91"/>
-<pinref part="J8" gate="G$1" pin="1"/>
-<wire x1="317.5" y1="55.88" x2="317.5" y2="50.8" width="0.1524" layer="91"/>
-<wire x1="317.5" y1="50.8" x2="322.58" y2="50.8" width="0.1524" layer="91"/>
-<junction x="317.5" y="55.88"/>
-</segment>
-</net>
+</segment>
+</net>
