File: pcb/led/led.brd (EAGLE design)
At the start: 305 x 244 mm, 181 parts, among them U2 USBC_16P

Commit message: atx rgb done, updated atx psu board too
Parts:
- added C27: 47uF, clock:C1210
- added JP2: (no value), pinhead:1X04
- added LED163: (no value), adafruit:CHIP-LED0805
- added R3, R4: 5.1K, joyAnalog:0805
- added R9: 1K, SparkFun-Passives:0805
- added U1: USBC_16P, my_usbc_16p:USBC_16P_FOOT
- LED148, LED21: device lul:REVERSE_MNT -> led:REVERSE_MNT
- moved LED6 27.1 mm to (89.9, 26.8)
- moved R1 20.9 mm to (99.5, 17.5)
- moved R2 20.9 mm to (99.5, 21.2)
- moved U2 20.9 mm to (107.4, 18.9)
- moved JP1 20.2 mm to (107.4, 28.0)
- moved LED7 19.5 mm to (139.7, 23.9)
- moved LED15 13.5 mm to (300.0, 14.0)
- moved LED23 11.7 mm to (104.0, 36.0), turned to 180 degrees
- moved LED24 11.4 mm to (80.6, 36.1), turned to 180 degrees
- moved LED22 10.8 mm to (129.0, 36.0), turned to 180 degrees
- moved LED5 10.5 mm to (84.8, 15.4), turned to 90 degrees
- moved LED3 9.13 mm to (47.5, 14.0)
- moved LED1 9.00 mm to (5.00, 14.0)
- moved LED10 9.00 mm to (195.0, 14.0)
- moved LED11 9.00 mm to (215.0, 14.0)
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Connections:
- removed net VDD: LED106.VDD, LED136.VDD, LED46.VDD, LED76.VDD
- new net N$166: JP1.2, U2.A7, U2.B7
- new net N$167: JP2.3, U1.A6, U1.B6
- new net N$168: JP2.2, LED162.DOUT, U1.A7, U1.B7
- new net N$170: LED163.C, R9.2
- new net N$7: R3.1, U1.A5
- net +5V: now also C27.1, JP1.4, JP2.4, LED106.VDD, LED136.VDD, LED163.A, LED46.VDD, LED76.VDD, U1.A4B9, U1.B4A9; no longer JP1.1
- net GND: now also C27.2, JP1.1, JP2.1, R3.2, R4.2, R9.1, U1.A1B12, U1.B11A12, U1.P$13, U1.P$14, U1.P$15, U1.P$16; no longer JP1.4
- net N$164: now also R4.1, U1.B5; no longer JP1.3, U2.A6, U2.B6
- net N$165: now also JP1.3, U2.A6, U2.B6; no longer JP1.2, U2.A7, U2.B7
Routing:
- net GND: track 2.95 -> 481.3 mm, vias 57 -> 162
- net N$168: track 0.00 -> 403.4 mm, vias 0 -> 1
- net +5V: track 4.87 -> 65.0 mm, vias 2 -> 28
- net N$6: track 24.0 -> 51.9 mm
- net N$24: track 51.3 -> 34.4 mm
- net N$21: track 56.4 -> 42.6 mm
- net N$14: track 10.4 -> 20.4 mm
- net N$7: track 0.00 -> 8.82 mm
- net N$167: track 0.00 -> 8.40 mm
- net N$18: track 50.3 -> 42.1 mm
- net N$166: track 0.00 -> 7.87 mm
- net N$15: track 21.0 -> 13.4 mm
- net N$23: track 24.7 -> 18.8 mm
- net N$5: track 15.4 -> 10.3 mm
- net N$44: track 20.8 -> 16.8 mm
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Other:
- outline, holes or cut-outs redrawn
- board text added: "5V"
- board text added: "DI"
- board text added: "DO"
- board text added: "GND"
- board text added: "PWR"
- board text added: "Pimp my Beeb ATX RGB Adaptor Plate dekuNukem SEPT 2022"
