File: pcb/led/led.sch (EAGLE design)
At the start: 181 parts, among them U2 USBC_16P

Commit message: atx rgb done, updated atx psu board too
Parts:
- added C27: 47uF, clock:C-USC1210
- added JP2: (no value), pinhead:PINHD-1X4
- added LED163: (no value), adafruit:LEDCHIP-LED0805
- added R3, R4: 5.1K, joyAnalog:RESISTOR0805-RES
- added R9: 1K, SparkFun-Passives:RESISTOR0805-RES
- added U1: USBC_16P, my_usbc_16p:USBC_16P
- LED148, LED21: device lul:WS2812B -> led:WS2812B
Connections:
- new net N$166: JP1.2, U2.DN1, U2.DN2
- new net N$167: JP2.3, U1.DP1, U1.DP2
- new net N$168: JP2.2, LED162.DO, U1.DN1, U1.DN2
- new net N$170: LED163.C, R9.2
- new net N$7: R3.1, U1.CC1
- net +5V: now also C27.1, JP1.4, JP2.4, LED106.VDD, LED136.VDD, LED163.A, LED46.VDD, LED76.VDD, U1.VBUS; no longer JP1.1
- net GND: now also C27.2, JP1.1, JP2.1, LED106.GND, LED19.GND, LED46.GND, R3.2, R4.2, R9.1, U1.GND; no longer JP1.4
- net N$164: now also R4.1, U1.CC2; no longer JP1.3, U2.DP1, U2.DP2
- net N$165: now also JP1.3, U2.DP1, U2.DP2; no longer JP1.2, U2.DN1, U2.DN2
