File: pcb/atx psu/atx_power_control.brd (EAGLE design)
At the start: 86 x 70 mm, 61 parts, among them IC2 REG1117, IC3 STM32F042F4, IC4 MY_7905DT, J1 ATX24RH, SW1 324_SW, SW2 324_SW, SW3 324_SW, SW4 324_SW, SW5 324_SW, SW6 324_SW, SW7 324_SW, U1 USBC_16P, U2 USBC_16P

Commit message: cleaned up files
Parts:
- moved SW1 0.54 mm to (25.1, 19.1)
- moved JP2 0.25 mm to (52.6, 50.0)
Other:
- board text removed: "MODE"
Changed lines of the file:
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@@
 <text x="77.724" y="43.942" size="1.9304" layer="25" rot="R90" align="center">5V</text>
 <text x="77.597" y="54.356" size="1.9304" layer="25" rot="R90" align="center">12V</text>
-<text x="56.6374" y="58.3908" size="1.4224" layer="25" rot="R270" align="center">GND</text>
-<text x="54.0974" y="58.3908" size="1.4224" layer="25" rot="R270" align="center">12V</text>
-<text x="51.5574" y="58.3908" size="1.4224" layer="25" rot="R270" align="center">SEN</text>
-<text x="49.0174" y="58.3908" size="1.4224" layer="25" rot="R270" align="center">PWM</text>
-<text x="23.876" y="25.146" size="1.4224" layer="25" rot="R180" align="center">HARD
+<text x="56.3834" y="58.3908" size="1.4224" layer="25" rot="R270" align="center">GND</text>
+<text x="53.8434" y="58.3908" size="1.4224" layer="25" rot="R270" align="center">12V</text>
+<text x="51.3034" y="58.3908" size="1.4224" layer="25" rot="R270" align="center">SEN</text>
+<text x="48.7634" y="58.3908" size="1.4224" layer="25" rot="R270" align="center">PWM</text>
+<text x="24.13" y="24.892" size="1.4224" layer="25" rot="R180" align="center">HARD
 PWR</text>
 <text x="30.734" y="24.892" size="1.4224" layer="25" rot="R180" align="center">SOFT
@@
 <circle x="4.318" y="65.786" radius="4" width="0" layer="42"/>
 <circle x="81.153" y="65.913" radius="4" width="0" layer="42"/>
-<text x="58.6278" y="34.925" size="2.1844" layer="25" rot="R270" align="center">FUSE 3A MAX</text>
+<text x="56.7228" y="36.195" size="2.54" layer="25" rot="R270" align="center">FUSE 3A MAX</text>
 <text x="77.724" y="58.7718" size="1.9304" layer="25" rot="R270" align="center">G</text>
 <text x="77.597" y="48.6118" size="1.9304" layer="25" rot="R270" align="center">G</text>
@@
 <text x="47.244" y="13.716" size="1.4224" layer="25" rot="R90" align="center">BRIGHT</text>
 <text x="49.784" y="13.716" size="1.4224" layer="25" rot="R270" align="center">FAN SPD</text>
-<text x="42.164" y="13.716" size="1.27" layer="25" rot="R270" align="center">RGB MODE</text>
+<text x="42.164" y="13.462" size="1.4224" layer="25" rot="R270" align="center">RGB MODE</text>
 <text x="25.8618" y="47.879" size="1.4224" layer="25" rot="R270" align="center">5VSB</text>
 <text x="22.2296" y="47.6542" size="1.4224" layer="25" rot="R90" align="center">PG</text>
 <text x="46.101" y="51.943" size="2.1844" layer="25" rot="R90" align="center">FAN</text>
 <text x="59.436" y="50.546" size="2.1844" layer="25" rot="R90" align="center">ARGB</text>
-<text x="37.592" y="25.019" size="1.27" layer="25" align="center">MODE</text>
+<text x="37.719" y="26.035" size="1.27" layer="25" align="center">RGB
+MODE</text>
 <text x="37.592" y="9.525" size="1.27" layer="25" align="center">COLOR</text>
 <text x="54.864" y="9.525" size="1.27" layer="25" rot="R180" align="center">BRIGHT</text>
@@
 <attribute name="VALUE" x="31.115" y="31.623" size="1.27" layer="27" rot="R180"/>
 </element>
-<element name="SW1" library="3pos_slide_switch_centered" package="342_SWICH_FOOT" value="324_SW" x="25.527" y="19.431" smashed="yes" rot="R270"/>
+<element name="SW1" library="3pos_slide_switch_centered" package="342_SWICH_FOOT" value="324_SW" x="25.146" y="19.05" smashed="yes" rot="R270"/>
 <element name="JP6" library="pinhead" library_urn="urn:adsk.eagle:library:325" package="1X02" package3d_urn="urn:adsk.eagle:package:22435/2" value="" x="30.988" y="19.812" smashed="yes" rot="R180">
 <attribute name="POPULARITY" value="98" x="30.988" y="19.812" size="1.778" layer="27" rot="R180" display="off"/>
@@
 <attribute name="VALUE" x="63.754" y="23.114" size="1.27" layer="27" rot="R180"/>
 </element>
-<element name="JP2" library="pinhead" library_urn="urn:adsk.eagle:library:325" package="1X04" package3d_urn="urn:adsk.eagle:package:22407/2" value="" x="52.832" y="50.038" smashed="yes">
-<attribute name="POPULARITY" value="91" x="52.832" y="50.038" size="1.778" layer="27" display="off"/>
-<attribute name="VALUE" x="47.752" y="46.863" size="1.27" layer="27"/>
+<element name="JP2" library="pinhead" library_urn="urn:adsk.eagle:library:325" package="1X04" package3d_urn="urn:adsk.eagle:package:22407/2" value="" x="52.578" y="50.038" smashed="yes">
+<attribute name="POPULARITY" value="91" x="52.578" y="50.038" size="1.778" layer="27" display="off"/>
+<attribute name="VALUE" x="47.498" y="46.863" size="1.27" layer="27"/>
 </element>
 <element name="JP7" library="pinhead" library_urn="urn:adsk.eagle:library:325" package="1X04" package3d_urn="urn:adsk.eagle:package:22407/2" value="" x="66.04" y="50.038" smashed="yes">
@@
 <wire x1="69.7865" y1="43.815" x2="72.461" y2="43.815" width="1.6764" layer="16"/>
 <wire x1="72.461" y1="43.815" x2="82.804" y2="54.158" width="1.6764" layer="16"/>
-<wire x1="54.102" y1="50.038" x2="54.102" y2="48.133" width="1.524" layer="16"/>
-<wire x1="58.42" y1="43.815" x2="64.7065" y2="43.815" width="1.524" layer="16"/>
-<wire x1="54.102" y1="48.133" x2="58.42" y2="43.815" width="1.524" layer="16"/>
+<wire x1="53.848" y1="50.038" x2="53.848" y2="48.133" width="1.524" layer="16"/>
+<wire x1="58.166" y1="43.815" x2="64.7065" y2="43.815" width="1.524" layer="16"/>
+<wire x1="53.848" y1="48.133" x2="58.166" y2="43.815" width="1.524" layer="16"/>
 </signal>
 <signal name="N$18">
@@
 <contactref element="SW1" pad="P$3"/>
 <wire x1="37.46" y1="31.5132" x2="37.46" y2="29.71285625" width="0.2032" layer="1"/>
-<wire x1="26.652" y1="17.231" x2="26.652" y2="19.812" width="1.016" layer="1"/>
+<wire x1="26.271" y1="16.85" x2="26.271" y2="19.812" width="1.016" layer="1"/>
 <contactref element="JP6" pad="2"/>
-<wire x1="26.652" y1="19.812" x2="26.652" y2="21.631" width="1.016" layer="1"/>
+<wire x1="26.271" y1="19.812" x2="26.271" y2="21.25" width="1.016" layer="1"/>
 <wire x1="29.718" y1="21.97085625" x2="37.46" y2="29.71285625" width="0.2032" layer="1"/>
 <wire x1="29.718" y1="19.812" x2="29.718" y2="21.97085625" width="0.2032" layer="1"/>
 <contactref element="J5" pad="1"/>
-<wire x1="29.718" y1="19.812" x2="26.652" y2="19.812" width="0.2032" layer="1"/>
-<wire x1="26.652" y1="17.231" x2="26.652" y2="14.75" width="0.2032" layer="1"/>
-<wire x1="26.652" y1="14.75" x2="29.21" y2="12.192" width="0.2032" layer="1"/>
+<wire x1="29.718" y1="19.812" x2="26.271" y2="19.812" width="0.2032" layer="1"/>
+<wire x1="26.271" y1="16.85" x2="26.271" y2="15.131" width="0.2032" layer="1"/>
+<wire x1="26.271" y1="15.131" x2="29.21" y2="12.192" width="0.2032" layer="1"/>
 </signal>
 <signal name="N$28">
@@
 <contactref element="JP2" pad="2"/>
 <contactref element="IC3" pad="12"/>
-<wire x1="54.991" y1="45.212" x2="51.562" y2="48.641" width="0.2032" layer="1"/>
-<wire x1="51.562" y1="50.038" x2="51.562" y2="48.641" width="0.2032" layer="1"/>
-<wire x1="54.991" y1="45.212" x2="54.991" y2="41.275" width="0.2032" layer="1"/>
+<wire x1="54.991" y1="44.958" x2="51.308" y2="48.641" width="0.2032" layer="1"/>
+<wire x1="51.308" y1="50.038" x2="51.308" y2="48.641" width="0.2032" layer="1"/>
+<wire x1="54.991" y1="44.958" x2="54.991" y2="41.275" width="0.2032" layer="1"/>
 <wire x1="54.991" y1="41.275" x2="52.451" y2="38.735" width="0.2032" layer="1"/>
 <wire x1="41.36" y1="38.185" x2="41.36" y2="37.3488" width="0.2032" layer="1"/>
@@
 <wire x1="41.402" y1="39.37" x2="43.307" y2="39.37" width="0.2032" layer="1"/>
 <wire x1="43.307" y1="39.37" x2="45.593" y2="41.656" width="0.2032" layer="1"/>
-<wire x1="45.593" y1="41.656" x2="45.593" y2="45.847" width="0.2032" layer="1"/>
-<wire x1="49.022" y1="49.276" x2="49.022" y2="50.038" width="0.2032" layer="1"/>
-<wire x1="49.022" y1="49.276" x2="45.593" y2="45.847" width="0.2032" layer="1"/>
+<wire x1="45.593" y1="41.656" x2="45.593" y2="46.101" width="0.2032" layer="1"/>
+<wire x1="48.768" y1="49.276" x2="48.768" y2="50.038" width="0.2032" layer="1"/>
+<wire x1="48.768" y1="49.276" x2="45.593" y2="46.101" width="0.2032" layer="1"/>
 </signal>
 <signal name="N$17">
