File: pcb/mac_se_se30/macse.sch (EAGLE design)
At the start: 9 parts, among them J2 ATX24RH

Commit message: finishing touches
Parts:
- added C1, C2: (no value), capacitor-wima:C5/2.5
Connections:
- net +12V: now also C1.1, C2.1
- net GND: now also C1.2, C2.2
Changed lines of the file:
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@@
 <part name="TP1" library="testpad" library_urn="urn:adsk.eagle:library:385" deviceset="PTR1" device="PAD1-20Y" package3d_urn="urn:adsk.eagle:package:27951/1"/>
 <part name="GND1" library="supply1" library_urn="urn:adsk.eagle:library:371" deviceset="GND" device=""/>
+<part name="P+4" library="supply1" library_urn="urn:adsk.eagle:library:371" deviceset="+12V" device=""/>
+<part name="GND5" library="supply1" library_urn="urn:adsk.eagle:library:371" deviceset="GND" device=""/>
+<part name="C2" library="capacitor-wima" library_urn="urn:adsk.eagle:library:116" deviceset="C" device="5/2.5" package3d_urn="urn:adsk.eagle:package:5426/1"/>
+<part name="C1" library="capacitor-wima" library_urn="urn:adsk.eagle:library:116" deviceset="C" device="5/2.5" package3d_urn="urn:adsk.eagle:package:5426/1"/>
 </parts>
 <sheets>
@@
 <instance part="GND1" gate="1" x="144.78" y="142.24" smashed="yes">
 <attribute name="VALUE" x="142.24" y="139.7" size="1.778" layer="96"/>
+</instance>
+<instance part="P+4" gate="1" x="20.32" y="144.78" smashed="yes" rot="MR0">
+<attribute name="VALUE" x="22.86" y="139.7" size="1.778" layer="96" rot="MR90"/>
+</instance>
+<instance part="GND5" gate="1" x="20.32" y="124.46" smashed="yes">
+<attribute name="VALUE" x="17.78" y="121.92" size="1.778" layer="96"/>
+</instance>
+<instance part="C2" gate="G$1" x="27.94" y="134.62" smashed="yes">
+<attribute name="NAME" x="29.464" y="135.001" size="1.778" layer="95"/>
+<attribute name="VALUE" x="29.464" y="129.921" size="1.778" layer="96"/>
+</instance>
+<instance part="C1" gate="G$1" x="20.32" y="134.62" smashed="yes">
+<attribute name="NAME" x="21.844" y="135.001" size="1.778" layer="95"/>
+<attribute name="VALUE" x="21.844" y="129.921" size="1.778" layer="96"/>
 </instance>
 </instances>
@@
 <wire x1="137.16" y1="144.78" x2="144.78" y2="144.78" width="0.1524" layer="91"/>
 </segment>
+<segment>
+<pinref part="GND5" gate="1" pin="GND"/>
+<wire x1="20.32" y1="129.54" x2="20.32" y2="127" width="0.1524" layer="91"/>
+<pinref part="C1" gate="G$1" pin="2"/>
+<pinref part="C2" gate="G$1" pin="2"/>
+<wire x1="27.94" y1="129.54" x2="20.32" y2="129.54" width="0.1524" layer="91"/>
+<junction x="20.32" y="129.54"/>
+</segment>
 </net>
 <net name="-12V" class="0">
@@
 <wire x1="-17.78" y1="134.62" x2="-7.62" y2="134.62" width="0.1524" layer="91"/>
 </segment>
-</net>
+<segment>
+<pinref part="P+4" gate="1" pin="+12V"/>
+<wire x1="20.32" y1="142.24" x2="20.32" y2="137.16" width="0.1524" layer="91"/>
+<pinref part="C1" gate="G$1" pin="1"/>
+<pinref part="C2" gate="G$1" pin="1"/>
+<wire x1="20.32" y1="137.16" x2="27.94" y2="137.16" width="0.1524" layer="91"/>
+<junction x="20.32" y="137.16"/>
+</segment>
+</net>
