File: pcb/pd1/atx4vc.sch (EAGLE design)
At the start: 76 parts, among them IC2 REG1117, IC3 STM32F042F4, IC4 MY_7905DT, J1 ATX24RH, SW1 324_SW, SW2 324_SW, SW3 324_SW, SW4 324_SW, SW5 324_SW, SW7 324_SW, U1 USBC_16P, U2 USBC_16P

Commit message: adding power connector and fuse detect
Parts:
- removed JP15: (no value), pinhead:PINHD-2X3
- removed R18, R19, R20, R21, R22: 5K1, atx_power_control:RESISTOR0805-RES
- removed U$4: VH396, 396_conn:VH396
- removed U$6: 74LVC2G08SSOP8, atx4vc:74LVC2G08SSOP8
- added JP8: (no value), atx_power_control:PINHD-1X4
- JP10: device adafruit:PINHD-1X1CB -> pinhead:PINHD-1X2
Connections:
- removed net N$24: JP3.2, U$6.3_2Y
- removed net N$38: IC3.PA3, JP3.1
- removed net N$39: R18.2, R19.1, U$6.7_1Y
- net +3V3: now also JP8.3; no longer JP15.5, U$6.8_VCC
- net GND: now also JP8.4; no longer JP15.6, R19.2, R20.2, R21.1, U$4.P$4, U$4.P$6, U$6.4_GND
- net N$11: no longer U$4.P$2
- net N$12: now also IC3.PA3, JP10.2; no longer U$6.1_1A, U$6.5_2A
- net N$15: no longer R18.1, U$4.P$7
- net N$16: no longer R21.2, U$4.P$3, U$6.2_1B
- net N$17: no longer R22.1
- net N$2: no longer U$4.P$1
- net N$3: now also JP8.1; no longer JP15.4
- net N$30: no longer R20.1, R22.2, U$4.P$5, U$6.6_2B
- net N$4: now also JP8.2; no longer JP15.3
- net PG: now also JP3.1
- net VCC: now also JP3.2
Other:
- moved on the sheet: JP3, R12
