File: pcb/appleii/appleii.brd (EAGLE design)
At the start: 75 x 47 mm, 17 parts, among them J1 POWER_JACKPTH, J2 ATX24RH

Commit message: working on appleii
Parts:
- removed JP3: (no value), atx_power_control:1X04
- added C5: (no value), capacitor-wima:C5B2.5
- added JP4: (no value), appleii:1X04
- JP1: device atx_power_control:1X04 -> appleii:1X04
- moved C3 8.68 mm to (2.03, 4.32)
- moved C4 8.46 mm to (2.03, 13.5)
- moved JP1 8.40 mm to (69.6, 5.84)
- moved U$4 1.32 mm to (62.0, 21.3)
- moved C1 0.90 mm to (50.8, 26.4), turned to 180 degrees
- moved U$8 0.84 mm to (45.0, 35.6)
- moved C2 0.56 mm to (39.4, 26.4), turned to 180 degrees
- moved J1 0.50 mm to (63.5, 47.0)
- moved U$2 0.42 mm to (45.0, 43.2)
- moved IC1 0.40 mm to (73.7, 32.0)
- moved J7 0.24 mm to (5.08, 33.3)
- moved JP2 0.23 mm to (5.59, 43.4)
- moved J2 0.11 mm to (30.5, 8.89)
Connections:
- net +12V: now also C1.+, JP1.2; no longer JP1.3
- net +5V: now also C2.+, JP4.2; no longer JP3.3
- net -5V: now also C5.1
- net GND: now also C1.-, C2.-, C3.2, C4.2, C5.2, JP1.1, JP4.1; no longer JP1.4, JP3.4
- net N$6: now also C4.1
- net N$8: now also C3.1
Routing:
- net N$8: track 0.00 -> 103.3 mm, vias 0 -> 1
- net N$6: track 0.00 -> 96.7 mm
- net +12V: track 0.00 -> 60.2 mm
- net +5V: track 0.00 -> 58.3 mm
- net -12V: track 0.00 -> 27.5 mm
- net N$5: track 0.00 -> 20.7 mm
- net -5V: track 0.00 -> 19.3 mm

Commit message: working on appleii
Parts:
- added U$7: VH396_2P, 396_conn:396_2P
- J1: device SparkFun:POWER_JACK_PTH -> appleii:POWER_JACK_PTH
- moved J1 1.02 mm to (62.5, 47.0)
- moved U$2 1.02 mm to (43.9, 43.2)
- moved U$8 1.02 mm to (43.9, 35.6)
- moved IC1 0.96 mm to (74.4, 31.4)
Connections:
- new net N$1: J1.PWR, U$7.P$2
- net GND: now also J1.GND, J1.GNDBREAK, U$7.P$1
Routing:
- net N$1: track 0.00 -> 12.7 mm
- net +5V: track 58.3 -> 56.3 mm
- net +12V: track 60.2 -> 61.2 mm
- net N$8: track 103.3 -> 102.3 mm
- net N$6: track 96.7 -> 96.1 mm
- net -5V: track 19.3 -> 19.8 mm
- net -12V: track 27.5 -> 28.0 mm
Other:
- outline, holes or cut-outs redrawn
- board text added: "Apple II / II Plus / IIe ATX Adaptor"
- board text added: "PT0 dekuNukem Nov 2022"
- board text added: "RED"
- board text removed: "Macintosh SE ATX Adaptor"
- board text removed: "NOTCH TOWARDS EDGE"
- board text removed: "PD1 dekuNukem Nov 2022"
- board text removed: "PWR SW"

Commit message: working on appleii
Parts:
- moved JP2 4.07 mm to (5.33, 39.4)
- moved J7 1.83 mm to (3.56, 34.3), turned to 270 degrees
- moved U$7 0.25 mm to (72.4, 42.6)
Routing:
- net N$5: track 20.7 -> 52.2 mm
Other:
- board text added: "GND"
- board text added: "PS_ON"
- board text added: "min 1uF"
Changed lines of the file:
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@@
 <text x="30.48" y="10.16" size="1.9304" layer="26" distance="35" rot="MR0" align="center">Apple II / II Plus / IIe ATX Adaptor</text>
 <text x="30.48" y="3.81" size="1.4224" layer="26" distance="30" rot="MR0" align="center">PT0 dekuNukem Nov 2022</text>
-<wire x1="71.225" y1="74.846" x2="71.225" y2="68.496" width="0.254" layer="21"/>
-<wire x1="71.86" y1="68.496" x2="78.972" y2="68.496" width="1.016" layer="21"/>
-<wire x1="82.274" y1="74.846" x2="82.274" y2="68.496" width="0.254" layer="21"/>
-<wire x1="82.274" y1="68.496" x2="79.226" y2="68.496" width="0.254" layer="21"/>
-<wire x1="89.005" y1="74.846" x2="89.005" y2="68.496" width="0.254" layer="21"/>
-<wire x1="89.64" y1="68.496" x2="96.752" y2="68.496" width="1.016" layer="21"/>
-<wire x1="99.8" y1="68.496" x2="97.133" y2="68.496" width="0.254" layer="21"/>
-<wire x1="99.927" y1="74.592" x2="99.927" y2="68.496" width="0.254" layer="21"/>
 <text x="43.91" y="43.095" size="1.9304" layer="26" distance="35" rot="MR0" align="center">FUSE
 5A MAX</text>
 <text x="72.041" y="37.6262" size="1.778" layer="25" distance="35" align="center">RED</text>
-<text x="81.925" y="67.184" size="2.1844" layer="25" distance="35" align="center">+</text>
-<text x="84.465" y="64.39" size="2.1844" layer="26" distance="35" rot="MR0" align="center">+</text>
 <circle x="2.5" y="22" radius="4" width="0" layer="41"/>
 <circle x="72.5" y="22" radius="4" width="0" layer="41"/>
@@
 <text x="53.467" y="24.003" size="2.1844" layer="25" distance="35" align="center">+</text>
 <wire x1="74.676" y1="46.736" x2="74.676" y2="39.116" width="1.016" layer="21"/>
+<text x="69.216" y="13.325" size="1.016" layer="25" distance="35" rot="R315" align="center">min 1uF</text>
+<text x="4.183" y="43.907" size="1.778" layer="25" rot="R270" align="center">GND</text>
+<text x="8.417" y="30.599" size="1.778" layer="25" align="center">GND</text>
+<text x="9.009" y="40.605" size="1.778" layer="25" rot="R270" align="center">PS_ON</text>
+<text x="9.687" y="34.409" size="1.778" layer="25" align="center">PS_ON</text>
 </plain>
 <attributes>
@@
 </autorouter>
 <elements>
-<element name="J7" library="atx_power_control" package="SCREWTERMINAL-3.5MM-2-NS" value="" x="5.08" y="33.274" smashed="yes" rot="R90">
-<attribute name="PROD_ID" value="CONN-13512" x="5.08" y="33.274" size="1.778" layer="27" rot="R90" display="off"/>
-<attribute name="SF_ID" value="PRT-09918" x="5.08" y="33.274" size="1.778" layer="27" rot="R90" display="off"/>
-<attribute name="SF_SKU" value="PRT-08432" x="5.08" y="33.274" size="1.778" layer="27" rot="R90" display="off"/>
-<attribute name="SKU" value="PRT-09914" x="5.08" y="33.274" size="1.778" layer="27" rot="R90" display="off"/>
-<attribute name="VALUE" x="3.81" y="32.004" size="0.6096" layer="27" font="vector" ratio="20" rot="R90"/>
+<element name="J7" library="atx_power_control" package="SCREWTERMINAL-3.5MM-2-NS" value="" x="3.556" y="34.29" smashed="yes" rot="R270">
+<attribute name="PROD_ID" value="CONN-13512" x="3.556" y="34.29" size="1.778" layer="27" rot="R270" display="off"/>
+<attribute name="SF_ID" value="PRT-09918" x="3.556" y="34.29" size="1.778" layer="27" rot="R270" display="off"/>
+<attribute name="SF_SKU" value="PRT-08432" x="3.556" y="34.29" size="1.778" layer="27" rot="R270" display="off"/>
+<attribute name="SKU" value="PRT-09914" x="3.556" y="34.29" size="1.778" layer="27" rot="R270" display="off"/>
+<attribute name="VALUE" x="4.826" y="35.56" size="0.6096" layer="27" font="vector" ratio="20" rot="R270"/>
 </element>
 <element name="U$8" library="atx_power_control" package="FUSE_HOLDER_3IN1" value="CAR_FUSE_HOLDER3IN1" x="43.942" y="35.56" smashed="yes" rot="R180"/>
 <element name="U$2" library="atx_power_control" package="FUSE_HOLDER_3IN1" value="CAR_FUSE_HOLDER3IN1" x="43.942" y="43.18" smashed="yes"/>
-<element name="JP2" library="pinhead" library_urn="urn:adsk.eagle:library:325" package="1X02" package3d_urn="urn:adsk.eagle:package:22435/2" value="" x="5.588" y="43.434" smashed="yes" rot="R180">
-<attribute name="POPULARITY" value="98" x="5.588" y="43.434" size="1.778" layer="27" rot="R180" display="off"/>
-<attribute name="VALUE" x="8.128" y="46.609" size="1.27" layer="27" rot="R180"/>
+<element name="JP2" library="pinhead" library_urn="urn:adsk.eagle:library:325" package="1X02" package3d_urn="urn:adsk.eagle:package:22435/2" value="" x="5.334" y="39.37" smashed="yes" rot="R180">
+<attribute name="POPULARITY" value="98" x="5.334" y="39.37" size="1.778" layer="27" rot="R180" display="off"/>
+<attribute name="VALUE" x="7.874" y="42.545" size="1.27" layer="27" rot="R180"/>
 </element>
 <element name="J2" library="macse" package="ATX24_RIGHT_ANGLE" value="ATX24RH" x="30.48" y="8.89" smashed="yes"/>
@@
 <element name="JP4" library="appleii" package="1X04" value="" x="61.468" y="5.842" smashed="yes" rot="R270"/>
 <element name="JP1" library="appleii" package="1X04" value="" x="69.596" y="5.842" smashed="yes" rot="R270"/>
-<element name="U$7" library="396_conn" package="396_2P" value="VH396_2P" x="72.136" y="42.5958" smashed="yes" rot="R270"/>
+<element name="U$7" library="396_conn" package="396_2P" value="VH396_2P" x="72.39" y="42.5958" smashed="yes" rot="R270"/>
 </elements>
 <signals>
@@
 <wire x1="40.98" y1="19.98" x2="37.846" y2="23.114" width="0.508" layer="16"/>
 <wire x1="27.398" y1="23.114" x2="27.398" y2="28.114" width="0.508" layer="16"/>
-<wire x1="5.08" y1="33.274" x2="6.858" y2="43.434" width="0" layer="19" extent="1-1"/>
-<wire x1="27.398" y1="28.114" x2="5.08" y2="33.274" width="0" layer="19" extent="1-1"/>
+<wire x1="21.222" y1="34.29" x2="6.604" y2="34.29" width="0.508" layer="1"/>
+<wire x1="6.604" y1="34.29" x2="3.556" y2="34.29" width="0.508" layer="1"/>
+<wire x1="27.398" y1="28.114" x2="21.222" y2="34.29" width="0.508" layer="1"/>
+<wire x1="6.604" y1="39.37" x2="6.604" y2="34.29" width="0.508" layer="1"/>
 </signal>
 <signal name="-5V">
@@
 <contactref element="U$7" pad="P$2"/>
 <wire x1="62.484" y1="33.29" x2="64.532" y2="33.29" width="3.175" layer="16"/>
-<wire x1="71.8578" y1="40.6158" x2="72.136" y2="40.6158" width="3.175" layer="16"/>
+<wire x1="71.8578" y1="40.6158" x2="72.39" y2="40.6158" width="3.175" layer="16"/>
 <wire x1="64.532" y1="33.29" x2="71.8578" y2="40.6158" width="3.175" layer="16"/>
 </signal>
