File: pcb/old/atx4vc.sch (EAGLE design)
At the start: 38 parts, among them IC4 MY_7905DT, J1 ATX24RH

Commit message: added 5VSB to terminal block, cleaned up files
Parts:
- removed J4: (no value), SparkFun-Connectors:USB_C16PIN
- removed JP2: (no value), pinhead:PINHD-1X2
- removed JP4: (no value), pinhead:PINHD-2X2
- removed U$11: M3_MOUNTING_HOLE, a:M3_MOUNTING_HOLE
- removed U$12: PINHD1X4, adafruit_changed:PINHD1X4
- added C1, C4: 100nF, atx_power_control:CAP0805
- added C2: 10uF, atx_power_control:CAP0805
- added IC2: REG1117, atx_power_control:REG1117
- added IC3: STM32F042F4, tx:STM32F042F4
- added J5, J8: (no value), atx_power_control:CONN_023.5MM
- added JP10: (no value), adafruit:PINHD-1X1CB
- added JP11: (no value), pinhead:PINHD-1X3
- added JP12: (no value), pinhead:PINHD-1X4
- added JP13: JUMPER-SMT_2_NO_NO-SILK, SparkFun-Jumpers:JUMPER-SMT_2_NO_NO-SILK
- added JP15: (no value), pinhead:PINHD-2X3
- added JP16: (no value), appleii:4PIN_FAN
- added JP5: (no value), atx_power_control:PINHD-1X3:1
- added JP6: (no value), atx_power_control:PINHD-1X2
- added JP9: (no value), atx_power_control:PINHD-2X4
- added LED8: (no value), adafruit:LEDCHIP-LED0805
- added R1, R14, R15, R18, R19, R2, R20, R21, R5: 5K1, atx_power_control:RESISTOR0805-RES
- added SW1, SW2, SW3, SW4, SW5, SW7: 324_SW, 3pos_slide_switch_centered:324_SW
- added U1, U2: USBC_16P, my_usbc_16p:USBC_16P
- J1: device nomcu:ATX24RH -> SparkFun-Connectors:ATX24RH
- JP3: device pinhead:PINHD-2X3 -> pinhead:PINHD-1X2
- U$6: value M3_MOUNTING_HOLE -> 74LVC2G08; device a:M3_MOUNTING_HOLE -> atx4vc:74LVC2G08
- U$9: value DG2204R-5.0 -> WAGO257-7; device atx4vc:DG2204R-5.0 -> atx4vc:WAGO257-7
Connections:
- removed net N$11: J1.PWR_OK, JP3.5, LED3.A
- removed net N$15: J1.PS_ON, JP2.2, JP3.6
- new net +3V3: C2.2, C4.2, IC2.VOUT, IC3.VDD, IC3.VDDA, JP15.5, JP9.4, SW4.1, SW4.4, U$6.8_VCC
- new net BUTTON1: IC3.NRST, SW3.2, SW3.3
- new net BUTTON2: IC3.BOOT0/PB8, JP9.3, R5.2, SW4.2, SW4.3
- new net F12V_DIV2: R18.2, R19.1, U$6.6_2B
- new net N$12: U$6.2_1B, U$6.3_2Y
- new net N$13: IC3.PA0, JP9.6, SW2.1, SW2.4
- new net N$19: LED8.A, R15.2
- new net N$22: IC3.PA1, JP9.8, SW5.1, SW5.4
- new net N$23: IC3.PA2, JP10.1
- new net N$24: JP3.2, U$6.7_1Y
- new net N$25: IC3.PF0/OSC_IN, J1.PS_ON, JP5.1, JP5.2
- new net N$26: IC3.PF1/OSC_OUT, J5.1, JP6.2, SW1.2, SW1.3
- new net N$27: IC3.PA4, JP9.2, SW7.1, SW7.4
- new net N$31: R1.1, U2.CC2
- new net N$33: R2.1, U2.CC1
- new net N$34: JP13.2, U1.DP1, U1.DP2
- new net N$35: IC3.PA7, JP12.2, JP13.1
- new net N$36: U1.DN1, U1.DN2
- new net N$38: IC3.PA3, JP3.1
- new net PG: IC3.PA10/PA12, J1.PWR_OK, JP15.1, LED3.A, U2.DP1, U2.DP2
- new net USB_DN: IC3.PA9/PA11, R15.1, U2.DN1, U2.DN2
- net -12V: now also U$9.P$1; no longer U$9.P$7
- net -5V: now also U$9.P$2; no longer U$9.P$6
- net F12V: now also JP16.2_VCC, R18.1, U$4.P$7, U$9.P$7; no longer U$4.P$5, U$9.P$3
- net F3V3: now also R21.2, U$6.1_1A, U$9.P$3; no longer U$9.P$5
- net F5V: now also JP12.1, R20.1, U$4.P$5, U$6.5_2A, U$9.P$5, U1.VBUS; no longer J4.VBUS, U$12.1, U$4.P$4, U$9.P$4
- net GND: now also C1.1, C2.1, C4.1, IC2.GND, IC3.VSS, J5.2, J8.1, JP11.3, JP12.4, JP15.6, JP16.1_GND, JP5.3, JP6.1, JP9.1, JP9.5, JP9.7, LED8.C, R1.2, R19.2, R2.2, R20.2, R21.1, R5.1, SW1.1, SW1.4, SW2.2, SW2.3, SW3.1, SW3.4, SW5.2, SW5.3, SW7.2, SW7.3, U$4.P$4, U$6.4_GND, U$9.P$4, U$9.P$6, U1.GND, U2.GND; no longer J4.GND, J4.SHLD, JP2.1, JP3.2, U$12.4, U$4.P$7, U$9.P$1, U$9.P$2
- net N$17: now also J8.2
- net N$3: now also IC3.PA14, JP15.4; no longer JP3.3, JP8.4_PWM
- net N$4: now also IC3.PA13, JP15.3; no longer J4.D+, JP4.2
- net N$6: now also IC3.PA6, JP11.1, R14.1; no longer J4.D-, JP4.4
- net N$7: now also IC3.PB1, JP16.4_PWM, JP8.4_PWM; no longer JP3.4, JP4.1, JP4.3, U$12.2
- net VCC: now also C1.2, IC2.VIN, JP11.2, JP15.2, R14.2, U2.VBUS; no longer JP3.1
Other:
- moved on the sheet: R12
