File: pcb/rev4/atx4vc.brd (EAGLE design)
At the start: 69 x 69 mm, 51 parts, among them IC1 MY_7905DT, IC2 MAX486X/SOT, J2 ATX24RH, SW1 SPST_TACT-EVQQ2

Commit message: finishing touches
Routing:
- net N$17: track 15.5 -> 14.4 mm
Other:
- board text added: "ATX4VC REV4 dekuNukem NOV24"
- board text removed: "ATX4VC REV4 dekuNukem MAY24"
Changed lines of the file:
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@@
 <grid distance="5" unitdist="mil" unit="mil" style="lines" multiple="1" display="no" altdistance="1" altunitdist="mil" altunit="mil"/>
 <layers>
-<layer number="1" name="Top" color="4" fill="1" visible="no" active="yes"/>
+<layer number="1" name="Top" color="4" fill="1" visible="yes" active="yes"/>
 <layer number="2" name="Route2" color="16" fill="1" visible="no" active="no"/>
 <layer number="3" name="Route3" color="17" fill="1" visible="no" active="no"/>
@@
 <layer number="19" name="Unrouted" color="6" fill="1" visible="yes" active="yes"/>
 <layer number="20" name="Dimension" color="24" fill="1" visible="yes" active="yes"/>
-<layer number="21" name="tPlace" color="7" fill="1" visible="no" active="yes"/>
+<layer number="21" name="tPlace" color="7" fill="1" visible="yes" active="yes"/>
 <layer number="22" name="bPlace" color="7" fill="1" visible="yes" active="yes"/>
-<layer number="23" name="tOrigins" color="15" fill="1" visible="no" active="yes"/>
+<layer number="23" name="tOrigins" color="15" fill="1" visible="yes" active="yes"/>
 <layer number="24" name="bOrigins" color="15" fill="1" visible="yes" active="yes"/>
-<layer number="25" name="tNames" color="7" fill="1" visible="no" active="yes"/>
+<layer number="25" name="tNames" color="7" fill="1" visible="yes" active="yes"/>
 <layer number="26" name="bNames" color="7" fill="1" visible="yes" active="yes"/>
-<layer number="27" name="tValues" color="7" fill="1" visible="no" active="yes"/>
-<layer number="28" name="bValues" color="7" fill="1" visible="no" active="yes"/>
+<layer number="27" name="tValues" color="7" fill="1" visible="yes" active="yes"/>
+<layer number="28" name="bValues" color="7" fill="1" visible="yes" active="yes"/>
 <layer number="29" name="tStop" color="7" fill="3" visible="no" active="yes"/>
 <layer number="30" name="bStop" color="7" fill="6" visible="no" active="yes"/>
@@
 <layer number="37" name="tTest" color="7" fill="1" visible="no" active="yes"/>
 <layer number="38" name="bTest" color="7" fill="1" visible="no" active="yes"/>
-<layer number="39" name="tKeepout" color="4" fill="11" visible="no" active="yes"/>
+<layer number="39" name="tKeepout" color="4" fill="11" visible="yes" active="yes"/>
 <layer number="40" name="bKeepout" color="1" fill="11" visible="yes" active="yes"/>
-<layer number="41" name="tRestrict" color="4" fill="10" visible="no" active="yes"/>
+<layer number="41" name="tRestrict" color="4" fill="10" visible="yes" active="yes"/>
 <layer number="42" name="bRestrict" color="1" fill="10" visible="yes" active="yes"/>
 <layer number="43" name="vRestrict" color="2" fill="10" visible="no" active="yes"/>
@@
 <layer number="49" name="Reference" color="7" fill="1" visible="no" active="yes"/>
 <layer number="50" name="dxf" color="7" fill="1" visible="no" active="no"/>
-<layer number="51" name="tDocu" color="7" fill="1" visible="no" active="yes"/>
+<layer number="51" name="tDocu" color="7" fill="1" visible="yes" active="yes"/>
 <layer number="52" name="bDocu" color="7" fill="1" visible="yes" active="yes"/>
 <layer number="53" name="tGND_GNDA" color="7" fill="1" visible="no" active="no"/>
@@
 <circle x="4.0355" y="64.931" radius="4" width="0" layer="42"/>
 <circle x="65.0705" y="65.058" radius="4" width="0" layer="42"/>
-<text x="83.3375" y="40.886" size="2.1844" layer="25" rot="R90" align="center">ATX4VC REV4
+<text x="32.901" y="24.4095" size="2.1844" layer="26" rot="MR0" align="center">ATX4VC REV4
 dekuNukem
-MAY24</text>
+NOV24</text>
 <wire x1="10.2145" y1="60.754" x2="58.9285" y2="60.754" width="0.0762" layer="20"/>
 <wire x1="58.9285" y1="60.754" x2="60.8335" y2="62.659" width="0.0762" layer="20" curve="90"/>
@@
 <dimension x1="65.0655" y1="65" x2="65.0655" y2="4" x3="94.5175" y3="34.5" textsize="1.778" layer="51" dtype="vertical"/>
 <text x="30.0175" y="46.4" size="1.6764" layer="26" rot="MR0" align="center">5V</text>
-<text x="35.5185" y="21.23" size="3.175" layer="26" ratio="10" rot="MR0" align="center">ATX4VC.com</text>
+<text x="37.0425" y="23.008" size="3.175" layer="25" ratio="10" align="center">ATX4VC.com</text>
 <hole x="9.017" y="61.087" drill="0.381"/>
 <hole x="60.325" y="61.087" drill="0.381"/>
@@
 </polygon>
 <contactref element="U$13" pad="2"/>
-<wire x1="46.6165" y1="11.3" x2="46.5515" y2="11.235" width="0.3048" layer="1"/>
 <wire x1="49.051" y1="10.639" x2="48.641" y2="11.049" width="0.3048" layer="1"/>
 <wire x1="61.3485" y1="10.639" x2="49.051" y2="10.639" width="0.3048" layer="1"/>
@@
 <contactref element="R3" pad="1"/>
 <contactref element="U$13" pad="1"/>
-<wire x1="58.8725" y1="14.942" x2="58.8725" y2="16.01" width="0.3048" layer="1"/>
 <wire x1="58.8725" y1="16.01" x2="58.8725" y2="14.4225" width="0.3048" layer="1"/>
 <wire x1="58.8725" y1="14.4225" x2="58.039" y2="13.589" width="0.3048" layer="1"/>
@@
 <contactref element="J2" pad="8"/>
 <contactref element="LED7" pad="A"/>
-<wire x1="11.1965" y1="40.8" x2="10.8155" y2="40.8" width="0.3048" layer="1"/>
 <contactref element="U$12" pad="P$16"/>
 <contactref element="U$12" pad="P$15"/>

Commit message: finishing touches
Parts:
- R3: value 470 -> 330
Changed lines of the file:
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@@
 <attribute name="NAME" x="57.033" y="43.95" size="0.8128" layer="25" rot="R90"/>
 </element>
-<element name="R3" library="atx_power_control" package="0805" value="470" x="46.6165" y="12.2" smashed="yes" rot="R270">
+<element name="R3" library="atx_power_control" package="0805" value="330" x="46.6165" y="12.2" smashed="yes" rot="R270">
 <attribute name="NAME" x="45.903" y="13.7875" size="0.8128" layer="25"/>
 </element>
